File: hw_drawings/straingauge.kicad_sch (KiCad schematic)
At the start: 105 parts, among them U1 AD7124-8BCPZ, U2 LT8333RDD-PBF, U3 LT3045xMSE, U4 LT3094xDD, U5 LT8333RDD-PBF, U6 Pico, U7 OPTO_DARL_6N138S, U8 LT3045xMSE, Y1 Crystal

Commit message: finished schematic
Parts:
- removed CR1: PMEG4020EPK_315, PMEG4020EPK-315:DIODE_DFN1608D-2_NEX, symbol 2024-04-24_11-49-29:PMEG4020EPK_315
- removed L2: 742792040, IND_742792040_WRE, symbol 2024-04-23_15-07-48:742792040
- removed U6: Pico, RPi_Pico:RPi_Pico_SMD_TH, symbol MCU_RaspberryPi_and_Boards:Pico
- removed U7: OPTO_DARL_6N138S, 8-SMD, symbol SparkFun-DiscreteSemi:OPTO_DARL_6N138S
- removed Y1: Crystal, symbol Device:Crystal
- added C29: 15p, Capacitor_SMD:C_0201_0603Metric, symbol Device:C
- added C30, C55: 1u, Capacitor_SMD:C_0603_1608Metric, symbol Device:C
- added C57: 4.7p, Capacitor_SMD:C_0402_1005Metric, symbol Device:C
- added CR3: PMEG4020EPK_315, PMEG4020EPK-315:DIODE_DFN1608D-2_NEX, symbol ShottKeyPmeg4020:PMEG4020EPK_315
- added J1: Conn_01x10_Pin, Connector_PinHeader_2.54mm:PinHeader_1x10_P2.54mm_Vertical, symbol Connector:Conn_01x10_Pin
- added J2, J3, J4, J5, J6, J7, J8, J9: Conn_01x06_Pin, Connector_PinHeader_2.54mm:PinHeader_1x06_P2.54mm_Vertical, symbol Connector:Conn_01x06_Pin
- added L2: 742792040, ul_7429:IND_742792040_WRE, symbol ferrite_bead:742792040
- added R23: 1k, Resistor_SMD:R_0805_2012Metric, symbol Device:R
- added R24: 2K, Resistor_SMD:R_0805_2012Metric, symbol Device:R
- added TP1, TP10, TP11, TP12, TP13, TP14, TP15, TP16, TP17, TP18, TP19, TP2, TP20, TP21, TP22, TP23, TP24, TP25, TP26, TP27, TP28, TP29, TP3, TP30, TP31, TP32, TP33, TP4, TP5, TP6, TP7, TP8, TP9: ~, TestPoint:TestPoint_Pad_1.5x1.5mm, symbol Connector:TestPoint
- added U6: Pico, RPi_Pico:RPi_Pico_SMD_TH, symbol RPi_Pico:Pico
- added U7: SI8380PM-IU, opto8bit:QSOP20_SIL, symbol opto8bit:SI8380PM-IU
- added U9: SIT8008BC-83-33E-2.4576, SIT8008BC-83-33E-10.000000_SIT, symbol 2-4576chmos:SIT8008BC-83-33E-2.4576
- C1, C13, C17, C24, C27, C33, C36, C39, C42, C45, C48, C50, C54: footprint (none) -> Capacitor_SMD:C_1206_3216Metric
- C10, C11, C12, C15, C16, C18, C20, C21, C5, C8: footprint (none) -> Capacitor_SMD:C_0603_1608Metric
- C14, C25, C28, C4: value 100n -> .1u; footprint (none) -> Capacitor_SMD:C_0603_1608Metric
- C19, C2: value 16u -> 10u; footprint (none) -> Capacitor_SMD:C_1206_3216Metric
- C22, C26, C31, C32, C34, C35, C37, C38, C40, C41, C43, C44, C46, C47, C49, C51, C52, C53, C7: footprint (none) -> Capacitor_SMD:C_0805_2012Metric
- C3, C6: footprint (none) -> Capacitor_SMD:C_0402_1005Metric
- C56: renamed from C?; footprint tant_68u:TAJB_AVX-L -> tant_68u:TAJB_AVX
- C9: footprint Capacitor_SMD:C_0201_0603Metric -> Capacitor_SMD:C_0603_1608Metric
- L1: footprint IND_XGL4020_COC -> xgl4020:IND_XGL4020_COC
- L3, L4: footprint IND_NFZ18SM121SN10D_MUR -> NFZ18SM121SN10D:IND_NFZ18SM121SN10D_MUR
- R1, R2, R3, R4: footprint Resistor_SMD:R_0603_1608Metric -> Resistor_SMD:R_0805_2012Metric
- R10, R11, R12, R13, R14, R15, R16, R17, R21, R22, R25, R26, R27, R28, R29, R30, R31, R32, R33, R34, R35, R36, R37, R38, R5, R6, R8, R9: footprint (none) -> Resistor_SMD:R_0805_2012Metric
- R18: value 1k -> 2.61k; footprint (none) -> Resistor_SMD:R_0805_2012Metric
- R19: value 5.1k -> 4.02k; footprint (none) -> Resistor_SMD:R_0805_2012Metric
- R20: value 3.9k -> 3.32k; footprint (none) -> Resistor_SMD:R_0805_2012Metric
- R7: value 70k -> 68k; footprint (none) -> Resistor_SMD:R_0805_2012Metric
- U1: footprint CP_32_12_ADI -> ad7124:CP_32_12_ADI
- U2, U5: footprint 05-08-1699_ADI -> LT83333:05-08-1699_ADI
Connections:
- net +3.3V: now also C55.1, R23.1, TP9.1, U9.4 (VDD)
- net +3.3VP: now also C30.1, U6.36 (3V3), U7.16 (VDD)
- net +5V: now also L2.1, TP21.1
- net +5VP: now also L2.2, U6.40 (VBUS)
- net -3.76v: now also C19.1, C20.1, C57.1, TP15.1; no longer C19.2, C20.2
- net -3v: now also J2.5 (Pin_5), J2.6 (Pin_6), J3.5 (Pin_5), J3.6 (Pin_6), J4.5 (Pin_5), J4.6 (Pin_6), J5.5 (Pin_5), J5.6 (Pin_6), J6.5 (Pin_5), J6.6 (Pin_6), J7.5 (Pin_5), J7.6 (Pin_6), J8.5 (Pin_5), J8.6 (Pin_6), J9.5 (Pin_5), J9.6 (Pin_6), TP1.1
- net 7.526v: now also CR3.1, TP16.1
- net 7v: now also J2.1 (Pin_1), J2.2 (Pin_2), J3.1 (Pin_1), J3.2 (Pin_2), J4.1 (Pin_1), J4.2 (Pin_2), J5.1 (Pin_1), J5.2 (Pin_2), J6.1 (Pin_1), J6.2 (Pin_2), J7.1 (Pin_1), J7.2 (Pin_2), J8.1 (Pin_1), J8.2 (Pin_2), J9.1 (Pin_1), J9.2 (Pin_2), TP2.1
- net GND: now also C19.2, C20.2, C21.2, C29.2, C30.2, C55.2, R24.2, TP28.1, TP29.1, U6.18 (GND), U7.15 (GND), U9.2 (GND); no longer C19.1, C20.1, C21.1
- net at U1.22 (REFOUT): now also TP12.1
- net at U1.25 (PSW): now also TP24.1
- net at U1.27 (*SYNC): now also TP23.1
- net at U1.28 (DOUT/*RDY): now also TP5.1, TP6.1, U6.21 (GPIO16)
- net at U1.29 (DIN): now also TP3.1, TP4.1, U6.25 (GPIO19)
- net at U1.30 (SCLK): now also TP33.1, U6.24 (GPIO18)
- net clock: now reaches U1.31 (CLK)
- net clock: now also C29.1, TP22.1, U9.3 (OUT)
- net at U1.32 (*CS): now also TP32.1, U6.22 (GPIO17)
- net at R21.2: now also J2.3 (Pin_3)
- net at R36.2: now also J8.4 (Pin_4)
- net at R26.2: now also J3.4 (Pin_4)
- net at C12.1, L3.1, U3.1 (IN)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: now also TP7.1
- net at R22.2: now also J2.4 (Pin_4)
- net at C7.1, R7.1, U3.8 (SET): now also R24.1
- net at C6.2, R1.2, R2.1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: now also TP14.1
- net at R37.2: now also J9.3 (Pin_3)
- net at R10.1, R11.2, U5.6 (FBX): now also C57.2, TP13.1
- net at R28.2: now also J4.4 (Pin_4)
- net at L1.1, U2.10 (SW): now also CR3.2
- net at R31.2: now also J6.3 (Pin_3)
- net at R25.2: now also J3.3 (Pin_3)
- net at R30.2: now also J5.4 (Pin_4)
- net at R27.2: now also J4.3 (Pin_3)
- net at R29.2: now also J5.3 (Pin_3)
- net at L4.1, U4.1 (IN), U4.3 (EN/UV): now also C21.1, TP8.1; no longer C21.2
- net at R32.2: now also J6.4 (Pin_4)
- net at R38.2: now also J9.4 (Pin_4)
- net at R34.2: now also J7.4 (Pin_4)
- net at R35.2: now also J8.3 (Pin_3)
- net at R33.2: now also J7.3 (Pin_3)
- net .9v renamed .3366v
- net .3366v: now also TP11.1
- net 1.9v renamed 2.959v
- net 2.959v: now also TP10.1
- new net: TP31.1, U6.14 (GPIO10)
- new net: TP30.1, U6.15 (GPIO11)
- new net: TP20.1, U6.16 (GPIO12)
- new net: TP19.1, U6.17 (GPIO13)
- new net: TP17.1, U6.19 (GPIO14)
- new net: TP18.1, U6.20 (GPIO15)
- new net: TP25.1, U6.41 (SWCLK)
- new net: TP26.1, U6.42 (GND)
- new net: TP27.1, U6.43 (SWDIO)
- new net: R23.2, U9.1 (OE/*ST/NC)
- new net: J1.1 (Pin_1), U7.1 (A1/AH1)
- new net: J1.10 (Pin_10), U7.10 (A8/AH8)
- new net: J1.2 (Pin_2), U7.2 (A2/AH2)
- new net: J1.3 (Pin_3), U7.3 (A3/AH3)
- new net: J1.4 (Pin_4), U7.4 (A4/AH4)
- new net: J1.5 (Pin_5), U7.5 (COM)
- new net: J1.6 (Pin_6), U7.6 (COM)
- new net: J1.7 (Pin_7), U7.7 (A5/AH5)
- new net: J1.8 (Pin_8), U7.8 (A6/AH6)
- new net: J1.9 (Pin_9), U7.9 (A7/AH7)
- new net opto0: U6.1 (GPIO0), U7.20 (B1/BH1)
- new net opto1: U6.2 (GPIO1), U7.19 (B2/BH2)
- new net opto2: U6.4 (GPIO2), U7.18 (B3/BH3)
- new net opto3: U6.5 (GPIO3), U7.17 (B4/BH4)
- new net opto4: U6.6 (GPIO4), U7.14 (B5/BH5)
- new net opto5: U6.7 (GPIO5), U7.13 (B6/BH6)
- new net opto6: U6.9 (GPIO6), U7.12 (B7/BH7)
- new net opto7: U6.10 (GPIO7), U7.11 (B8/BH8)
Other:
- moved on the sheet: C7, U1B

Commit message: pcb1
Parts:
- removed J2, J3, J4, J5, J6, J7, J8, J9: Conn_01x06_Pin, Connector_PinHeader_2.54mm:PinHeader_1x06_P2.54mm_Vertical, symbol Connector:Conn_01x06_Pin
- removed L1: XGL4020-152MEC, xgl4020:IND_XGL4020_COC, symbol 2024-04-23_13-18-42:XGL4020-152MEC
- removed TP25, TP26, TP27: ~, TestPoint:TestPoint_Pad_1.5x1.5mm, symbol Connector:TestPoint
- added D1, D10, D11, D12, D13, D14, D15, D16, D2, D3, D4, D5, D6, D7, D8, D9: BAT54S, Package_TO_SOT_SMD:SOT-23, symbol Diode:BAT54S
- added J2, J3, J4, J5, J6, J7, J8, J9: Conn_01x04_Pin, Connector_PinHeader_2.54mm:PinHeader_1x04_P2.54mm_Vertical, symbol Connector:Conn_01x04_Pin
- added L1: XGL4020-152MEC, xgl4020:IND_XGL4020_COC, symbol coicraftXGL4020MEC:XGL4020-152MEC
- C36, C42, C48: value 100n -> 10n; footprint Capacitor_SMD:C_1206_3216Metric -> Capacitor_SMD:C_0805_2012Metric
- C38, C44, C53: value 10n -> 100n; footprint Capacitor_SMD:C_0805_2012Metric -> Capacitor_SMD:C_1206_3216Metric
- R21, R22, R25, R26, R27, R28, R29, R30, R31, R32, R33, R34, R35, R36, R37, R38: value 1k -> 100
- U1: footprint ad7124:CP_32_12_ADI -> CP_32_12_ADI
- U2: footprint LT83333:05-08-1699_ADI -> 05-08-1699_ADI
- U6: now not fitted
Connections:
- net 7v is gone; now on net +7V: C17.1, R19.1, R5.1, TP2.1, U3.10 (OUTS), U3.11 (OUT)
- net +3.3V: now also U8.12 (OUT), D1.2 (K), D10.2 (K), D11.2 (K), D12.2 (K), D13.2 (K), D14.2 (K), D15.2 (K), D16.2 (K), D2.2 (K), D3.2 (K), D4.2 (K), D5.2 (K), D6.2 (K), D7.2 (K), D8.2 (K), D9.2 (K)
- net +5V: now also C12.1, C21.1, L3.1, L4.1, TP7.1, TP8.1, U3.1 (IN), U3.2 (IN), U3.3 (IN), U3.4 (EN/UV), U4.1 (IN), U4.13 (IN), U4.2 (IN), U4.3 (EN/UV), U8.2 (IN), U8.3 (IN), L1.2
- net -3v: now also U4.12 (OUT), J2.3 (Pin_3), J3.3 (Pin_3), J4.3 (Pin_3), J5.3 (Pin_3), J6.3 (Pin_3), J7.3 (Pin_3), J8.3 (Pin_3), J9.3 (Pin_3)
- net GND: now also C36.2, C37.1, C42.2, C43.1, C48.2, C52.1, U3.13 (GND), U6.38 (GND), U8.13 (GND), D1.1 (A), D10.1 (A), D11.1 (A), D12.1 (A), D13.1 (A), D14.1 (A), D15.1 (A), D16.1 (A), D2.1 (A), D3.1 (A), D4.1 (A), D5.1 (A), D6.1 (A), D7.1 (A), D8.1 (A), D9.1 (A); no longer C37.2, C38.1, C43.2, C44.1, C52.2, C53.1, U4.2 (IN)
- net AIN6: now reaches C41.2, R32.1, U1.10 (AIN6/IOUT/VBIAS)
- net AIN6: now also C44.1; no longer C42.1
- net AIN0: now reaches C54.1, R38.1, U1.4 (AIN0/IOUT/VBIAS)
- net AIN0: now also C52.2; no longer C53.2
- net AIN7: now reaches C40.1, R31.1, U1.11 (AIN7/IOUT/VBIAS)
- net AIN7: now also C44.2; no longer C42.2
- net AIN8: now reaches C39.1, R30.1, U1.14 (AIN8/IOUT/VBIAS)
- net AIN8: now also C37.2; no longer C38.2
- net AIN9: now reaches C39.2, R29.1, U1.15 (AIN9/IOUT/VBIAS)
- net AIN9: now also C36.1; no longer C37.1
- net AIN10: now reaches C35.2, R28.1, U1.16 (AIN10/IOUT/VBIAS)
- net AIN10: now also C38.1; no longer C36.1
- net AIN11: now reaches C34.1, R27.1, U1.17 (AIN11/IOUT/VBIAS)
- net AIN11: now also C38.2; no longer C36.2
- net AIN12: now reaches C32.2, C33.1, R26.1, U1.18 (AIN12/IOUT/VBIAS)
- net AIN13: now reaches C31.1, C33.2, R25.1, U1.19 (AIN13/IOUT/VBIAS)
- net AIN14: now reaches C49.2, C50.1, R22.1, U1.20 (AIN14/IOUT/VBIAS/REFIN2(+))
- net AIN15: now reaches C50.2, C51.1, R21.1, U1.21 (AIN15/IOUT/VBIAS/REFIN2(-))
- net AIN1: now reaches C54.2, R37.1, U1.5 (AIN1/IOUT/VBIAS)
- net AIN1: now also C48.1; no longer C52.1
- net AIN2: now reaches C47.2, R36.1, U1.6 (AIN2/IOUT/VBIAS/P1)
- net AIN2: now also C53.1; no longer C48.1
- net AIN3: now reaches C46.1, R35.1, U1.7 (AIN3/IOUT/VBIAS/P2)
- net AIN3: now also C53.2; no longer C48.2
- net AIN4: now reaches C45.1, R34.1, U1.8 (AIN4/IOUT/VBIAS/P3)
- net AIN4: now also C43.2; no longer C44.2
- net AIN5: now reaches C45.2, R33.1, U1.9 (AIN5/IOUT/VBIAS/P4)
- net AIN5: now also C42.1; no longer C43.1
- net at R21.2: now also D1.3 (COM), J2.2 (Pin_2)
- net at R22.2: now also D2.3 (COM), J2.1 (Pin_1)
- net at R36.2: now also D15.3 (COM), J8.1 (Pin_1)
- net at R26.2: now also D4.3 (COM), J3.1 (Pin_1)
- net at CR3.2, U2.10 (SW): now also L1.1
- net +7V: now reaches U3.12 (OUT)
- net +7V: now also J2.4 (Pin_4), J3.4 (Pin_4), J4.4 (Pin_4), J5.4 (Pin_4), J6.4 (Pin_4), J7.4 (Pin_4), J8.4 (Pin_4), J9.4 (Pin_4)
- net at R37.2: now also D14.3 (COM), J9.2 (Pin_2)
- net at R38.2: now also D16.3 (COM), J9.1 (Pin_1)
- net at R33.2: now also D10.3 (COM), J7.2 (Pin_2)
- net at R34.2: now also D12.3 (COM), J7.1 (Pin_1)
- net at R25.2: now also D3.3 (COM), J3.2 (Pin_2)
- net at R27.2: now also D5.3 (COM), J4.2 (Pin_2)
- net at R28.2: now also D7.3 (COM), J4.1 (Pin_1)
- net at R31.2: now also D9.3 (COM), J6.2 (Pin_2)
- net at R30.2: now also D8.3 (COM), J5.1 (Pin_1)
- net at R29.2: now also D6.3 (COM), J5.2 (Pin_2)
- net at R35.2: now also D13.3 (COM), J8.2 (Pin_2)
- net at R32.2: now also D11.3 (COM), J6.1 (Pin_1)
- net clock renamed CLK
- no-connect marks 0 -> 25
Other:
- company: (none) -> Utrecht university
- title: (none) -> ADC converter strain gauge
- moved on the sheet: C29, C49, C5, C50, C51, R2, R21, R22, R23, U9

Commit message: fixed ERC
Parts:
- removed TP7: ~, TestPoint:TestPoint_Pad_1.5x1.5mm, symbol Connector:TestPoint
- added C58: .1u, Capacitor_SMD:C_0603_1608Metric, symbol Device:C
- added R39, R40, R41, R42, R43, R44, R45, R46, R47, R48: 620, Resistor_SMD:R_0805_2012Metric, symbol Device:R
- U5: footprint LT83333:05-08-1699_ADI -> 05-08-1699_ADI
Connections:
- net +3.3V: now also U3.10 (OUTS), U3.11 (OUT), U3.12 (OUT); no longer U8.10 (OUTS), U8.11 (OUT), U8.12 (OUT)
- net +3.3VP: now also C58.1
- net +5V: now also C13.1, U5.1 (EN/UVLO); no longer C12.1, C21.1, L3.1, L4.1, TP8.1, U4.1 (IN), U4.13 (IN), U4.2 (IN), U4.3 (EN/UV), U8.1 (IN), U8.2 (IN), U8.3 (IN), U8.4 (EN/UV)
- net +7V: now also U8.10 (OUTS), U8.11 (OUT), U8.12 (OUT); no longer U3.10 (OUTS), U3.11 (OUT), U3.12 (OUT)
- net GND: now also C22.1, C58.2
- net at R5.2, R6.1: now also U8.7 (PGFB); no longer U3.7 (PGFB)
- net at R16.2, R17.1: now also U3.7 (PGFB); no longer U8.7 (PGFB)
- net at C26.1, R15.1: now also U3.8 (SET); no longer U8.8 (SET)
- net at C7.1, R24.1, R7.1: now also U8.8 (SET); no longer U3.8 (SET)
- net at U7.1 (A1/AH1): now also R39.2; no longer J1.1 (Pin_1)
- net at U7.10 (A8/AH8): now also R48.2; no longer J1.10 (Pin_10)
- net at U7.2 (A2/AH2): now also R40.2; no longer J1.2 (Pin_2)
- net at J1.3 (Pin_3): now also R41.1; no longer U7.3 (A3/AH3)
- net at U7.4 (A4/AH4): now also R42.2; no longer J1.4 (Pin_4)
- net at U7.5 (COM): now also R43.2; no longer J1.5 (Pin_5)
- net at U7.6 (COM): now also R44.2; no longer J1.6 (Pin_6)
- net at U7.7 (A5/AH5): now also R45.2; no longer J1.7 (Pin_7)
- net at U7.8 (A6/AH6): now also R46.2; no longer J1.8 (Pin_8)
- net at J1.9 (Pin_9): now also R47.1; no longer U7.9 (A7/AH7)
- net at C22.2, R12.2: now also U4.8 (SET)
- new net: R47.2, U7.9 (A7/AH7)
- new net: R41.2, U7.3 (A3/AH3)
- new net: J1.6 (Pin_6), R44.1
- new net: J1.10 (Pin_10), R48.1
- new net: J1.4 (Pin_4), R42.1
- new net: J1.8 (Pin_8), R46.1
- new net: J1.7 (Pin_7), R45.1
- new net: J1.1 (Pin_1), R39.1
- new net: J1.5 (Pin_5), R43.1
- new net: J1.2 (Pin_2), R40.1
- new net in3: C21.1, L4.1, TP8.1, U4.1 (IN), U4.13 (IN), U4.2 (IN), U4.3 (EN/UV)
- new net in7: C12.1, L3.1, U8.1 (IN), U8.2 (IN), U8.3 (IN), U8.4 (EN/UV)
Other:
- moved on the sheet: C14, C15, C16, C18, C19, C20, C21, C22, C23, C57, CR2, J1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

Commit message: supplies
Parts:
- added C59, C60, C61: 10u, Capacitor_SMD:C_1206_3216Metric, symbol Device:C
Connections:
- net +5V: now also C61.1
- net GND: now also C59.2, C60.2, C61.2
- net in3: now also C60.1
- net in7: now also C59.1

Commit message: ADC
Parts:
- removed J2, J3, J5, J6, J7, J8, J9: Conn_01x04_Pin, Connector_PinHeader_2.54mm:PinHeader_1x04_P2.54mm_Vertical, symbol Connector:Conn_01x04_Pin
- removed TP17, TP18, TP19, TP20, TP30, TP31: ~, TestPoint:TestPoint_Pad_1.5x1.5mm, symbol Connector:TestPoint
- added C62: .1u, Capacitor_SMD:C_0603_1608Metric, symbol Device:C
- added J2, J3: Conn_01x08_Pin, Connector_PinSocket_2.54mm:PinSocket_1x08_P2.54mm_Vertical, symbol Connector:Conn_01x08_Pin
Connections:
- net +3.3V: now also C62.1; no longer D9.2 (K)
- net +7V: now also J4.3 (Pin_3)
- net -3v: now also J4.1 (Pin_1), J4.2 (Pin_2); no longer J4.3 (Pin_3)
- net .3366v: no longer R18.2, R20.1, TP11.1, U1.13 (REFIN1(-))
- net 2.959v: no longer R18.1, R19.2, TP10.1, U1.12 (REFIN1(+))
- net AIN0: now also D16.3 (COM)
- net AIN1: now also D14.3 (COM)
- net AIN10: now also D7.3 (COM)
- net AIN11: now also D5.3 (COM)
- net AIN12: now also D4.3 (COM)
- net AIN13: now also D3.3 (COM)
- net AIN14: now also D2.3 (COM)
- net AIN15: now also D1.3 (COM)
- net AIN2: now also D15.3 (COM)
- net AIN3: now also D13.3 (COM)
- net AIN4: now also D12.3 (COM)
- net AIN5: now also D10.3 (COM)
- net AIN6: now also D11.3 (COM)
- net AIN7: now also D9.3 (COM)
- net AIN8: now also D8.3 (COM)
- net AIN9: now also D6.3 (COM)
- net GND: now also C62.2
- net DOUT/*RDY: now reaches TP5.1, TP6.1, U1.28 (DOUT/*RDY), U6.21 (GPIO16)
- net DIN: now reaches TP3.1, TP4.1, U1.29 (DIN), U6.25 (GPIO19)
- net SCLK: now reaches TP33.1, U1.30 (SCLK), U6.24 (GPIO18)
- net *CS: now reaches TP32.1, U1.32 (*CS), U6.22 (GPIO17)
- net at R38.2: now also J3.5 (Pin_5); no longer D16.3 (COM)
- net at R21.2: now also J2.8 (Pin_8); no longer D1.3 (COM)
- net at R33.2: now also J3.2 (Pin_2); no longer D10.3 (COM)
- net at R25.2: now also J2.6 (Pin_6); no longer D3.3 (COM)
- net at R37.2: now also J3.6 (Pin_6); no longer D14.3 (COM)
- net at R22.2: now also J2.7 (Pin_7); no longer D2.3 (COM)
- net at R32.2: now also J3.3 (Pin_3); no longer D11.3 (COM)
- net at R31.2: now also J3.4 (Pin_4); no longer D9.3 (COM)
- net at R26.2: now also J2.5 (Pin_5); no longer D4.3 (COM)
- net at R30.2: now also J2.1 (Pin_1); no longer D8.3 (COM)
- net at R29.2: now also J2.2 (Pin_2); no longer D6.3 (COM)
- net at R34.2: now also J3.1 (Pin_1); no longer D12.3 (COM)
- net at R36.2: now also J3.7 (Pin_7); no longer D15.3 (COM)
- net at R35.2: now also J3.8 (Pin_8); no longer D13.3 (COM)
- new net: J2.3 (Pin_3), R28.2
- new net: J2.4 (Pin_4), R27.2
- new net REFIN1(+): R18.1, R19.2, TP10.1, U1.12 (REFIN1(+))
- new net REFIN1(-): R18.2, R20.1, TP11.1, U1.13 (REFIN1(-))
Other:
- moved on the sheet: C25, C28, C29, C31, C32, C33, C34, C35, C36, C37, C38, C39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

Commit message: full pcb
Parts:
- removed J4: Conn_01x04_Pin, Connector_PinHeader_2.54mm:PinHeader_1x04_P2.54mm_Vertical, symbol Connector:Conn_01x04_Pin
- removed TP3, TP5, TP8: ~, TestPoint:TestPoint_Pad_1.5x1.5mm, symbol Connector:TestPoint
- added J4, J5: Conn_01x01_Pin, Connector_PinHeader_2.54mm:PinHeader_1x01_P2.54mm_Vertical, symbol Connector:Conn_01x01_Pin
- J2, J3: now not fitted
- renumbered TP15 to -3.8v, TP1 to -3v, TP11 to .33v, TP10 to 2.95v, TP9 to 33v, TP21 to 5v, TP16 to 7.5v, TP2 to 7v, TP32 to CS, TP4 to DIN, TP6 to DOUT, TP13 to FBX3, TP14 to FBX7, TP12 to FEF, TP24 to PSW, TP33 to SCLK, TP23 to SYNC, TP29 to gnd, TP28 to gnd
Connections:
- net +3.3V: now also D9.2 (K)
- net +7V: now also J4.1 (Pin_1)
- net -3v: now also J5.1 (Pin_1)

Commit message: full pcb1
Parts:
- renumbered -3.8v to -3.8v1, -3v to -3v1, .33v to .33v1, 2.95v to 2.95v1, 33v to 33v1, 5v to 5v1, 7.5v to 7.5v1, 7v to 7v1, CS to CS1, DIN to DIN1, DOUT to DOUT1, FEF to FEF1, PSW to PSW1, SCLK to SCLK1, SYNC to SYNC1, gnd to gnd1, gnd to gnd2
Connections:
- net GND: now also U6.23 (GND), U6.3 (GND), U6.8 (GND)
- no-connect marks 25 -> 28
Other:
- note added: ".3366v"
- note added: "2.959v"
- moved on the sheet: SCLK1

Commit message: full pcb1
Parts:
- removed -3v1, .33v1, 2.95v1, 7v1: ~, TestPoint:TestPoint_Pad_1.5x1.5mm, symbol Connector:TestPoint
- removed C56: 68u, tant_68u:TAJB_AVX, symbol Tantalum_68u:TAJB686K010RNJ
- removed U3, U8: LT3045xMSE, Package_SO:MSOP-12-1EP_3x4mm_P0.65mm_EP1.65x2.85mm, symbol Regulator3045:LT3045xMSE
- added C56: 47u, Resistor_SMD:R_1206_3216Metric, symbol Device:C
- added R49: 300, Resistor_SMD:R_0805_2012Metric, symbol Device:R
- added R50: 10, Resistor_SMD:R_0805_2012Metric, symbol Device:R
- added TP1, TP2: ~, TestPoint:TestPoint_Pad_1.5x1.5mm, symbol Connector:TestPoint
- added U10, U11: LT3045xDD, Package_DFN_QFN:DFN-10-1EP_3x3mm_P0.5mm_EP1.65x2.38mm, symbol Regulator_Linear_bb:LT3045xDD
- C1, C13, C17, C19, C2, C24, C27, C59, C60, C61: footprint Capacitor_SMD:C_1206_3216Metric -> Capacitor_SMD:C_0805_2012Metric
- C15, C30, C5, C55, C8, C9: footprint Capacitor_SMD:C_0603_1608Metric -> Capacitor_SMD:C_0402_1005Metric
- C29: footprint Capacitor_SMD:C_0201_0603Metric -> Capacitor_SMD:C_0402_1005Metric
- C3: footprint Capacitor_SMD:C_0402_1005Metric -> Capacitor_SMD:C_0603_1608Metric
- J4, J5: value Conn_01x01_Pin -> Pin
- R17: value 110k -> 100k
- R18: value 2.61k -> 240
- R19: value 4.02k -> 430
- R20: value 3.32k -> 10
- R39, R40, R41, R42, R45, R46, R47, R48: value 620 -> 680
- R43: value 620 -> 10k
- R44: value 620 -> 10
Connections:
- net +3.3V: now also U10.10 (OUT), U10.9 (OUTS)
- net +5V: now also C56.1, U10.1 (IN), U10.2 (IN), U10.3 (EN/UV)
- net +7V: now also U11.10 (OUT), U11.9 (OUTS)
- net GND: now also R43.1, C56.2, U10.11 (GND), U10.5 (ILIM), U10.8 (GND), U11.11 (GND), U11.5 (ILIM), U11.8 (GND); no longer R17.2
- net REFIN1(+): now also R44.2, TP1.1; no longer R19.2
- net REFIN1(-): now also R49.1, R50.2, TP2.1; no longer R18.2, R20.1
- net in7: now also U11.1 (IN), U11.2 (IN), U11.3 (EN/UV)
- net at R5.2, R6.1: now also U11.6 (PGFB)
- net at C7.1, R24.1, R7.1: now also U11.7 (SET)
- net at U7.5 (COM): now also J1.5 (Pin_5); no longer R43.2
- net at U7.6 (COM): now also J1.6 (Pin_6); no longer R44.2
- net at R44.1: now also R19.2; no longer J1.6 (Pin_6)
- net at C26.1, R15.1: now also U10.7 (SET)
- net at R17.1: now also R43.2; no longer R16.2
- new net: R20.1, R49.2
- new net: R18.2, R50.1
- new net: R16.2, R17.2, U10.6 (PGFB)
Other:
- note added: "100mV"
- note added: "2.6v"
- note removed: ".3366v"
- note removed: "2.959v"
- moved on the sheet: C17, C26, C7, R15, R16, R17, R18, R19, R20, R24, R5, R6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
