File: hw_drawings/straingauge.kicad_sch (KiCad schematic)
At the start: 167 parts, among them J1 Conn_01x10_Pin, J2 Conn_01x08_Pin, J3 Conn_01x08_Pin, J4 Pin, J5 Pin, U1 AD7124-8BCPZ, U10 LT3045xDD, U11 LT3045xDD, U2 LT8333RDD-PBF, U4 LT3094xDD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

Commit message: finished project
Parts:
- added D17: BAV99, Package_TO_SOT_SMD:SOT-23, symbol Diode:BAV99
- added H1, H2, H3, H4: MountingHole_Pad, MountingHole:MountingHole_3.2mm_M3_Pad, symbol Mechanical:MountingHole_Pad
- added R51: 680, Resistor_SMD:R_0805_2012Metric, symbol Device:R
- added R52: 16k, Resistor_SMD:R_0805_2012Metric, symbol Device:R
- C1, C13, C17, C19, C2, C24, C27, C59, C60, C61: LCSC (none) -> C15850
- C10, C14, C18, C25, C28, C4, C58, C62: LCSC (none) -> C14663
- C11, C12, C20, C21: LCSC (none) -> C377773
- C15, C30, C5, C55, C8, C9: LCSC (none) -> C52923
- C16: LCSC (none) -> C1595
- C22, C26, C7: LCSC (none) -> C1779
- C23: value tdk-1u -> 1u; footprint CAP_2012_TDK -> Capacitor_SMD:C_0402_1005Metric; LCSC (none) -> C52923
- C29: LCSC (none) -> C1548
- C3: LCSC (none) -> C1630
- C31, C32, C34, C35, C36, C37, C40, C41, C42, C43, C46, C47, C48, C49, C51, C52: LCSC (none) -> C441760
- C33, C38, C39, C44, C45, C50, C53, C54: LCSC (none) -> C338082
- C56: LCSC (none) -> C96123
- C57, C6: LCSC (none) -> C1569
- CR2, CR3: LCSC (none) -> C2999988
- D1, D10, D11, D12, D13, D14, D15, D16, D2, D3, D4, D5, D6, D7, D8, D9: LCSC (none) -> C727126
- L2: footprint ul_7429:IND_742792040_WRE -> IND_742792040_WRE; LCSC (none) -> C2661857
- L3, L4: LCSC (none) -> C338244
- R1, R10, R13, R16, R5: LCSC (none) -> C17514
- R11, R2: LCSC (none) -> C17589
- R12: LCSC (none) -> C17621
- R14: LCSC (none) -> C17436
- R15: LCSC (none) -> C17633
- R17: LCSC (none) -> C149504
- R18: LCSC (none) -> C17572
- R19: LCSC (none) -> C17695
- R20, R44, R50: LCSC (none) -> C17415
- R21, R22, R25, R26, R27, R28, R29, R30, R31, R32, R33, R34, R35, R36, R37, R38: LCSC (none) -> C17408
- R23: LCSC (none) -> C17513
- R24: LCSC (none) -> C17604
- R3, R7: LCSC (none) -> C17801
- R39, R40, R41, R42, R45, R46, R47, R48: LCSC (none) -> C17798
- R4, R8: LCSC (none) -> C4328
- R43: LCSC (none) -> C17414
- R49: LCSC (none) -> C17630
- R6: LCSC (none) -> C17713
- R9: LCSC (none) -> C25826
- U1: LCSC (none) -> C97314
- U10, U11: LCSC (none) -> C666574
- U2, U5: LCSC (none) -> C673740
- U4: LCSC (none) -> C670492
- U7: LCSC (none) -> C7315580
Connections:
- net +7V: now also D17.2 (A)
- net -3v: now also D17.1 (K)
- net GND: now also D17.3 (K), H1.1, H2.1, H3.1, H4.1, R51.2, R52.2; no longer U11.5 (ILIM), U4.6 (ILIM)
- net AIN0_C: now reaches R38.2
- net AIN0_C: now also J3.1 (Pin_1); no longer J3.5 (Pin_5)
- net AIN15_C: now reaches J2.8 (Pin_8), R21.2
- net AIN4_C: now reaches R34.2
- net AIN4_C: now also J3.5 (Pin_5); no longer J3.1 (Pin_1)
- net AIN1_C: now reaches J3.2 (Pin_2)
- net AIN1_C: now also R37.2; no longer R33.2
- net AIN2_C: now reaches J3.3 (Pin_3)
- net AIN2_C: now also R36.2; no longer R32.2
- net AIN3_C: now reaches J3.4 (Pin_4)
- net AIN3_C: now also R35.2; no longer R31.2
- net AIN5_C: now reaches J3.6 (Pin_6)
- net AIN5_C: now also R33.2; no longer R37.2
- net AIN6_C: now reaches J3.7 (Pin_7)
- net AIN6_C: now also R32.2; no longer R36.2
- net AIN7_C: now reaches J3.8 (Pin_8)
- net AIN7_C: now also R31.2; no longer R35.2
- net AIN14_C: now reaches J2.7 (Pin_7), R22.2
- net AIN12_C: now reaches J2.5 (Pin_5), R26.2
- net AIN13_C: now reaches J2.6 (Pin_6), R25.2
- net AIN10_C: now reaches J2.3 (Pin_3), R28.2
- net AIN11_C: now reaches J2.4 (Pin_4), R27.2
- net AIN9_C: now reaches J2.2 (Pin_2), R29.2
- net AIN8_C: now reaches J2.1 (Pin_1), R30.2
- new net: R52.1, U4.6 (ILIM)
- new net: R51.1, U11.5 (ILIM)
Other:
- note added: "150mA*kΩ: 220mA"
- note added: "3.75A*kΩ: 243mA"
- note removed: "max ~10uF total"
- moved on the sheet: C25, C28, C29, C40, C41, C42, C43, C44, C45, C46, C47, C48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

Commit message: changed bead
Parts:
- removed L2: 742792040, IND_742792040_WRE, symbol ferrite_bead:742792040
- removed L3, L4: NFZ18SM121SN10D, NFZ18SM121SN10D:IND_NFZ18SM121SN10D_MUR, symbol MurataNFZ18SM121SN10D:NFZ18SM121SN10D
- added FB1: 500 2A, Inductor_SMD:L_1206_3216Metric, symbol Device:FerriteBead
- added FB2, FB3: 120 1A, Inductor_SMD:L_0603_1608Metric, symbol Device:FerriteBead
Connections:
- net +5V: now also FB1.2
- net +5VP: now also FB1.1
- net -3.76v: now also FB3.1
- net 7.526v: now also FB2.1
- net in3: now also FB3.2
- net in7: now also FB2.2

Commit message: move l5
Parts:
- FB1: LCSC C515371 -> C2844587
- FB2, FB3: footprint Inductor_SMD:L_0603_1608Metric -> Inductor_SMD:L_0805_2012Metric; LCSC C2983009 -> C2844587
Changed lines of the file:
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@@
 			)
 		)
-		(property "Footprint" "Inductor_SMD:L_0603_1608Metric"
+		(property "Footprint" "Inductor_SMD:L_0805_2012Metric"
 			(at 152.4 142.748 90)
 			(effects
@@
 			)
 		)
-		(property "Description" "PB1608-121/1A0 "
+		(property "Description" "MLB2012F-101T"
 			(at 152.4 140.97 0)
 			(effects
@@
 			)
 		)
-		(property "LCSC" "C2983009"
+		(property "LCSC" "C2844587"
 			(at 152.4 140.97 0)
 			(effects
@@
 			)
 		)
-		(property "LCSC" "C515371"
+		(property "LCSC" "C2844587"
 			(at 39.37 25.4 0)
 			(effects
@@
 		(on_board yes)
 		(dnp no)
-		(fields_autoplaced yes)
 		(property "Reference" "FB2"
-			(at 152.3492 66.04 90)
+			(at 149.86 71.12 90)
 			(effects
 				(font
@@
 			)
 		)
-		(property "Footprint" "Inductor_SMD:L_0603_1608Metric"
+		(property "Footprint" "Inductor_SMD:L_0805_2012Metric"
 			(at 152.4 75.438 90)
 			(effects
@@
 			)
 		)
-		(property "Description" "PB1608-121/1A0 "
+		(property "Description" "MLB2012F-101T"
 			(at 152.4 73.66 0)
 			(effects
@@
 			)
 		)
-		(property "LCSC" "C2983009"
+		(property "LCSC" "C2844587"
 			(at 152.4 73.66 0)
 			(effects

Commit message: redesign
Parts:
- removed C14: .1u, Capacitor_SMD:C_0603_1608Metric, symbol Device:C
- removed C16: 1.5n, Capacitor_SMD:C_0603_1608Metric, symbol Device:C
- removed C23: 1u, Capacitor_SMD:C_0402_1005Metric, symbol TDK-1u50vcer:CGJ4J3X7R1H105K125AB
- removed C26: 4.7u, Capacitor_SMD:C_0805_2012Metric, symbol Device:C
- removed C27: 10u, Capacitor_SMD:C_0805_2012Metric, symbol Device:C
- removed CR2, CR3: PMEG4020EPK_315, PMEG4020EPK-315:DIODE_DFN1608D-2_NEX, symbol ShottKeyPmeg4020:PMEG4020EPK_315
- removed R15: 33k, Resistor_SMD:R_0805_2012Metric, symbol Device:R
- removed R16: 1M, Resistor_SMD:R_0805_2012Metric, symbol Device:R
- removed R17: 100k, Resistor_SMD:R_0805_2012Metric, symbol Device:R
- removed R3: 68k, Resistor_SMD:R_0805_2012Metric, symbol Device:R
- removed R4, R8: 20k, Resistor_SMD:R_0805_2012Metric, symbol Device:R
- removed R43: 10k, Resistor_SMD:R_0805_2012Metric, symbol Device:R
- removed R9: 39k, Resistor_SMD:R_0805_2012Metric, symbol Device:R
- removed U10: LT3045xDD, Package_DFN_QFN:DFN-10-1EP_3x3mm_P0.5mm_EP1.65x2.38mm, symbol Regulator_Linear_bb:LT3045xDD
- removed U2, U5: LT8333RDD-PBF, 05-08-1699_ADI, symbol lt8333:LT8333RDD-PBF
- added D18, D19: 1N5819WS, Diode_SMD:D_SOD-323, symbol Device:D_Schottky
- added U2, U3: LT8330ES6, TSOT-23_S6_LIT, symbol lt8330:LT8330ES6-TRMPBF
- added U5: AMS1117-3.3, Package_TO_SOT_SMD:SOT-223-3_TabPin2, symbol Regulator_Linear:AMS1117-3.3
- C3: value 680p -> 1u; footprint Capacitor_SMD:C_0603_1608Metric -> Capacitor_SMD:C_0402_1005Metric; LCSC C1630 -> C52923
- C4: value .1u -> 1u; footprint Capacitor_SMD:C_0603_1608Metric -> Capacitor_SMD:C_0402_1005Metric; LCSC C14663 -> C52923
- FB1: LCSC C2844587 -> C515371
- H1, H2, H3, H4: footprint MountingHole:MountingHole_3.2mm_M3_Pad -> MountingHole:MountingHole_2.2mm_M2
Connections:
- net +3.3V: now also C3.1, C30.1, U1.2 (IOVDD), U5.2 (VO)
- net +3.3VP: no longer C30.1, U1.2 (IOVDD)
- net +5V: now also U2.4 (EN/UVLO), U2.6 (VIN), U3.4 (EN/UVLO), U3.6 (VIN), U5.3 (VI)
- net 7.526v: now also D18.1 (K)
- net GND: now also C15.1, C5.1, D19.1 (K), U2.2 (GND), U3.2 (GND), U5.1 (GND); no longer C15.2, C4.2, C5.2
- net at C57.2, FBX3.1, R10.1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: now also U3.3 (FBX)
- net at L1.1: now also D18.2 (A), U2.1 (SW)
- net at C6.2, FBX7.1, R1.2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: now also U2.3 (FBX)
- net at L5.4: now also C4.2, D19.2 (A)
- net at L5.3: now also C4.1, U3.1 (SW)
- new net: C15.2, U3.5 (INTVCC)
- new net: C5.2, U2.5 (INTVCC)
- no-connect marks 28 -> 27
Other:
- moved on the sheet: -3.8v1, 7.5v1, C1, C10, C11, C12, C13, C15, C17, C18, C19, C2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
