File: hw_drawings/straingauge.kicad_pcb (KiCad board)
At the start: 2 copper layers, 153 parts, among them J1 Conn_01x10_Pin, J2 Conn_01x06_Pin, J3 Conn_01x06_Pin, J4 Conn_01x06_Pin, J5 Conn_01x06_Pin, J6 Conn_01x06_Pin, J7 Conn_01x06_Pin, J8 Conn_01x06_Pin, J9 Conn_01x06_Pin, U1 AD7124-8BCPZ, U2 LT8333RDD-PBF, U3 LT3045xMSE, U4 LT3094xDD, U5 LT8333RDD-PBF, U6 Pico, U7 SI8380PM-IU, U8 LT3045xMSE, U9 SIT8008BC-83-33E-2.4576

Commit message: pcb1
Parts:
- removed CR1: PMEG4020EPK_315, PMEG4020EPK-315:DIODE_DFN1608D-2_NEX
- removed TP25, TP26, TP27: ~, TestPoint:TestPoint_Pad_1.5x1.5mm
- added CR3: PMEG4020EPK_315, PMEG4020EPK-315:DIODE_DFN1608D-2_NEX, F.Cu at (125.1, 39.0)
- added D1: BAT54S, Package_TO_SOT_SMD:SOT-23, F.Cu at (242.4, 62.6)
- added D10: BAT54S, Package_TO_SOT_SMD:SOT-23, F.Cu at (252.2, 67.2)
- added D11: BAT54S, Package_TO_SOT_SMD:SOT-23, F.Cu at (252.2, 71.9)
- added D12: BAT54S, Package_TO_SOT_SMD:SOT-23, F.Cu at (252.2, 76.5)
- added D13: BAT54S, Package_TO_SOT_SMD:SOT-23, F.Cu at (257.1, 62.6)
- added D14: BAT54S, Package_TO_SOT_SMD:SOT-23, F.Cu at (257.1, 67.2)
- added D15: BAT54S, Package_TO_SOT_SMD:SOT-23, F.Cu at (257.1, 71.9)
- added D16: BAT54S, Package_TO_SOT_SMD:SOT-23, F.Cu at (257.1, 76.5)
- added D2: BAT54S, Package_TO_SOT_SMD:SOT-23, F.Cu at (242.4, 67.2)
- added D3: BAT54S, Package_TO_SOT_SMD:SOT-23, F.Cu at (242.4, 71.9)
- added D4: BAT54S, Package_TO_SOT_SMD:SOT-23, F.Cu at (242.4, 76.5)
- added D5: BAT54S, Package_TO_SOT_SMD:SOT-23, F.Cu at (247.3, 62.6)
- added D6: BAT54S, Package_TO_SOT_SMD:SOT-23, F.Cu at (247.3, 67.2)
- added D7: BAT54S, Package_TO_SOT_SMD:SOT-23, F.Cu at (247.3, 71.9)
- added D8: BAT54S, Package_TO_SOT_SMD:SOT-23, F.Cu at (247.3, 76.5)
- added D9: BAT54S, Package_TO_SOT_SMD:SOT-23, F.Cu at (252.2, 62.6)
- C36, C42, C48: value 100n -> 10n; footprint Capacitor_SMD:C_1206_3216Metric -> Capacitor_SMD:C_0805_2012Metric
- C38, C44, C53: value 10n -> 100n; footprint Capacitor_SMD:C_0805_2012Metric -> Capacitor_SMD:C_1206_3216Metric
- J2, J3, J4, J5, J6, J7, J8, J9: value Conn_01x06_Pin -> Conn_01x04_Pin; footprint Connector_PinHeader_2.54mm:PinHeader_1x06_P2.54mm_Vertical -> Connector_PinHeader_2.54mm:PinHeader_1x04_P2.54mm_Vertical
- R21, R22, R25, R26, R27, R28, R29, R30, R31, R32, R33, R34, R35, R36, R37, R38: value 1k -> 100
- U6: footprint MCU_RaspberryPi_and_Boards:RPi_Pico_SMD_TH -> RPi_Pico:RPi_Pico_SMD_TH
- moved R14 150.2 mm to (200.6, 99.0)
- moved R15 150.2 mm to (200.6, 102.0)
- moved R16 150.2 mm to (200.6, 104.9)
- moved R6 150.2 mm to (196.2, 99.0)
- moved R7 150.2 mm to (196.2, 102.0)
- moved R8 150.2 mm to (196.2, 104.9)
- moved R22 150.2 mm to (205.0, 99.0)
- moved R23 150.2 mm to (205.0, 102.0)
- moved R24 150.2 mm to (205.0, 104.9)
- moved R30 150.2 mm to (209.4, 99.0)
- moved R31 150.2 mm to (209.4, 102.0)
- moved R32 150.2 mm to (209.4, 104.9)
- moved R10 148.5 mm to (201.1, 78.5)
- moved R11 148.5 mm to (201.1, 81.5)
- moved R12 148.5 mm to (201.1, 84.5)
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Connections:
- net /clock renamed /CLK
- net Net-(U1A-AIN12/IOUT/VBIAS) renamed /AIN12
- net Net-(U1A-AIN13/IOUT/VBIAS) renamed /AIN13
- net Net-(U1A-AIN14/IOUT/VBIAS/REFIN2(+)) renamed /AIN14
- net Net-(U1A-AIN15/IOUT/VBIAS/REFIN2(-)) renamed /AIN15
- C12 pad 1: Net-(U3-EN/UV) -> +5V
- C17 pad 1: /7v -> +7V
- C21 pad 1: Net-(U4-EN/UV) -> +5V
- C24 pad 1: /-3v -> -3v
- C34 pad 1: Net-(U1A-AIN11/IOUT/VBIAS) -> /AIN11
- C35 pad 2: Net-(U1A-AIN10/IOUT/VBIAS) -> /AIN10
- C36 pad 1: Net-(U1A-AIN10/IOUT/VBIAS) -> /AIN9
- C36 pad 2: Net-(U1A-AIN11/IOUT/VBIAS) -> GND
- C37 pad 1: Net-(U1A-AIN9/IOUT/VBIAS) -> GND
- C37 pad 2: GND -> /AIN8
- C38 pad 1: GND -> /AIN10
- C38 pad 2: Net-(U1A-AIN8/IOUT/VBIAS) -> /AIN11
- C39 pad 1: Net-(U1A-AIN8/IOUT/VBIAS) -> /AIN8
- C39 pad 2: Net-(U1A-AIN9/IOUT/VBIAS) -> /AIN9
- C40 pad 1: Net-(U1A-AIN7/IOUT/VBIAS) -> /AIN7
- C41 pad 2: Net-(U1A-AIN6/IOUT/VBIAS) -> /AIN6
- C42 pad 1: Net-(U1A-AIN6/IOUT/VBIAS) -> /AIN5
- C42 pad 2: Net-(U1A-AIN7/IOUT/VBIAS) -> GND
- C43 pad 1: Net-(U1A-AIN5/IOUT/VBIAS/P4) -> GND
- C43 pad 2: GND -> /AIN4
- C44 pad 1: GND -> /AIN6
- C44 pad 2: Net-(U1A-AIN4/IOUT/VBIAS/P3) -> /AIN7
- C45 pad 1: Net-(U1A-AIN4/IOUT/VBIAS/P3) -> /AIN4
- C45 pad 2: Net-(U1A-AIN5/IOUT/VBIAS/P4) -> /AIN5
- C46 pad 1: Net-(U1A-AIN3/IOUT/VBIAS/P2) -> /AIN3
- C47 pad 2: Net-(U1A-AIN2/IOUT/VBIAS/P1) -> /AIN2
- C48 pad 1: Net-(U1A-AIN2/IOUT/VBIAS/P1) -> /AIN1
- C48 pad 2: Net-(U1A-AIN3/IOUT/VBIAS/P2) -> GND
- C52 pad 1: Net-(U1A-AIN1/IOUT/VBIAS) -> GND
- C52 pad 2: GND -> /AIN0
- C53 pad 1: GND -> /AIN2
- C53 pad 2: Net-(U1A-AIN0/IOUT/VBIAS) -> /AIN3
- C54 pad 1: Net-(U1A-AIN0/IOUT/VBIAS) -> /AIN0
- C54 pad 2: Net-(U1A-AIN1/IOUT/VBIAS) -> /AIN1
- J2 pad 1: /7v -> Net-(D2-COM)
- J2 pad 2: /7v -> Net-(D1-COM)
- J2 pad 3: Net-(J2-Pin_3) -> -3v
- J2 pad 4: Net-(J2-Pin_4) -> +7V
- J3 pad 1: /7v -> Net-(D4-COM)
- J3 pad 2: /7v -> Net-(D3-COM)
- J3 pad 3: Net-(J3-Pin_3) -> -3v
- J3 pad 4: Net-(J3-Pin_4) -> +7V
- J4 pad 1: /7v -> Net-(D7-COM)
- J4 pad 2: /7v -> Net-(D5-COM)
- J4 pad 3: Net-(J4-Pin_3) -> -3v
- J4 pad 4: Net-(J4-Pin_4) -> +7V
- J5 pad 1: /7v -> Net-(D8-COM)
- J5 pad 2: /7v -> Net-(D6-COM)
- J5 pad 3: Net-(J5-Pin_3) -> -3v
- J5 pad 4: Net-(J5-Pin_4) -> +7V
- J6 pad 1: /7v -> Net-(D11-COM)
- J6 pad 2: /7v -> Net-(D9-COM)
- J6 pad 3: Net-(J6-Pin_3) -> -3v
- J6 pad 4: Net-(J6-Pin_4) -> +7V
- J7 pad 1: /7v -> Net-(D12-COM)
- J7 pad 2: /7v -> Net-(D10-COM)
- J7 pad 3: Net-(J7-Pin_3) -> -3v
- J7 pad 4: Net-(J7-Pin_4) -> +7V
- J8 pad 1: /7v -> Net-(D15-COM)
- J8 pad 2: /7v -> Net-(D13-COM)
- J8 pad 3: Net-(J8-Pin_3) -> -3v
- J8 pad 4: Net-(J8-Pin_4) -> +7V
- J9 pad 1: /7v -> Net-(D16-COM)
- J9 pad 2: /7v -> Net-(D14-COM)
- J9 pad 3: Net-(J9-Pin_3) -> -3v
- J9 pad 4: Net-(J9-Pin_4) -> +7V
- L3 pad 1: Net-(U3-EN/UV) -> +5V
- L4 pad 1: Net-(U4-EN/UV) -> +5V
- R13 pad 2: /-3v -> -3v
- R19 pad 1: /7v -> +7V
- R20 pad 2: /-3v -> -3v
- R21 pad 2: Net-(J2-Pin_3) -> Net-(D1-COM)
- R22 pad 2: Net-(J2-Pin_4) -> Net-(D2-COM)
- R25 pad 2: Net-(J3-Pin_3) -> Net-(D3-COM)
- R26 pad 2: Net-(J3-Pin_4) -> Net-(D4-COM)
- R27 pad 1: Net-(U1A-AIN11/IOUT/VBIAS) -> /AIN11
- R27 pad 2: Net-(J4-Pin_3) -> Net-(D5-COM)
- R28 pad 1: Net-(U1A-AIN10/IOUT/VBIAS) -> /AIN10
- R28 pad 2: Net-(J4-Pin_4) -> Net-(D7-COM)
- R29 pad 1: Net-(U1A-AIN9/IOUT/VBIAS) -> /AIN9
- R29 pad 2: Net-(J5-Pin_3) -> Net-(D6-COM)
- R30 pad 1: Net-(U1A-AIN8/IOUT/VBIAS) -> /AIN8
- R30 pad 2: Net-(J5-Pin_4) -> Net-(D8-COM)
- R31 pad 1: Net-(U1A-AIN7/IOUT/VBIAS) -> /AIN7
- R31 pad 2: Net-(J6-Pin_3) -> Net-(D9-COM)
- R32 pad 1: Net-(U1A-AIN6/IOUT/VBIAS) -> /AIN6
- R32 pad 2: Net-(J6-Pin_4) -> Net-(D11-COM)
- R33 pad 1: Net-(U1A-AIN5/IOUT/VBIAS/P4) -> /AIN5
- R33 pad 2: Net-(J7-Pin_3) -> Net-(D10-COM)
- R34 pad 1: Net-(U1A-AIN4/IOUT/VBIAS/P3) -> /AIN4
- R34 pad 2: Net-(J7-Pin_4) -> Net-(D12-COM)
- R35 pad 1: Net-(U1A-AIN3/IOUT/VBIAS/P2) -> /AIN3
- R35 pad 2: Net-(J8-Pin_3) -> Net-(D13-COM)
- R36 pad 1: Net-(U1A-AIN2/IOUT/VBIAS/P1) -> /AIN2
- R36 pad 2: Net-(J8-Pin_4) -> Net-(D15-COM)
- R37 pad 1: Net-(U1A-AIN1/IOUT/VBIAS) -> /AIN1
- R37 pad 2: Net-(J9-Pin_3) -> Net-(D14-COM)
- R38 pad 1: Net-(U1A-AIN0/IOUT/VBIAS) -> /AIN0
- R38 pad 2: Net-(J9-Pin_4) -> Net-(D16-COM)
- R5 pad 1: /7v -> +7V
- TP1 pad 1: /-3v -> -3v
- TP2 pad 1: /7v -> +7V
- TP7 pad 1: Net-(U3-EN/UV) -> +5V
- TP8 pad 1: Net-(U4-EN/UV) -> +5V
- U1 pad 10: Net-(U1A-AIN6/IOUT/VBIAS) -> /AIN6
- U1 pad 11: Net-(U1A-AIN7/IOUT/VBIAS) -> /AIN7
- U1 pad 14: Net-(U1A-AIN8/IOUT/VBIAS) -> /AIN8
- U1 pad 15: Net-(U1A-AIN9/IOUT/VBIAS) -> /AIN9
- U1 pad 16: Net-(U1A-AIN10/IOUT/VBIAS) -> /AIN10
- U1 pad 17: Net-(U1A-AIN11/IOUT/VBIAS) -> /AIN11
- U1 pad 4: Net-(U1A-AIN0/IOUT/VBIAS) -> /AIN0
- U1 pad 5: Net-(U1A-AIN1/IOUT/VBIAS) -> /AIN1
- U1 pad 6: Net-(U1A-AIN2/IOUT/VBIAS/P1) -> /AIN2
- U1 pad 7: Net-(U1A-AIN3/IOUT/VBIAS/P2) -> /AIN3
- U1 pad 8: Net-(U1A-AIN4/IOUT/VBIAS/P3) -> /AIN4
- U1 pad 9: Net-(U1A-AIN5/IOUT/VBIAS/P4) -> /AIN5
- U3 pad 1: Net-(U3-EN/UV) -> +5V
- U3 pad 10: /7v -> +7V
- U3 pad 11: /7v -> +7V
- U3 pad 12: unconnected-(U3-OUT-Pad12) -> +7V
- U3 pad 13: unconnected-(U3-GND-Pad13) -> GND
- U3 pad 2: unconnected-(U3-IN-Pad2) -> +5V
- U3 pad 3: unconnected-(U3-IN-Pad3) -> +5V
- U3 pad 4: Net-(U3-EN/UV) -> +5V
- U4 pad 1: Net-(U4-EN/UV) -> +5V
- U4 pad 10: /-3v -> -3v
- U4 pad 11: /-3v -> -3v
- U4 pad 12: unconnected-(U4-OUT-Pad12) -> -3v
- U4 pad 13: unconnected-(U4-IN-Pad13) -> +5V
- U4 pad 2: GND -> +5V
- U4 pad 3: Net-(U4-EN/UV) -> +5V
- U6 pad 38: unconnected-(U6-GND-Pad38) -> GND
- U6 pad 41: Net-(U6-SWCLK) -> unconnected-(U6-SWCLK-Pad41)
- U6 pad 42: Net-(TP26-Pad1) -> unconnected-(U6-GND-Pad42)_0
- U6 pad 43: Net-(U6-SWDIO) -> unconnected-(U6-SWDIO-Pad43)
- U8 pad 12: unconnected-(U8-OUT-Pad12) -> +3.3V
- U8 pad 13: unconnected-(U8-GND-Pad13) -> GND
- U8 pad 2: unconnected-(U8-IN-Pad2) -> +5V
- U8 pad 3: unconnected-(U8-IN-Pad3) -> +5V
Routing:
- net +5V: track 0.00 -> 61.5 mm, vias 0 -> 6
- net GND: track 0.00 -> 29.9 mm, vias 0 -> 14
- net +5VP: track 0.00 -> 21.5 mm, vias 0 -> 3
- net /7.526v: track 0.00 -> 7.93 mm
- net Net-(U2-FBX): track 0.00 -> 7.68 mm
- net Net-(U2-SW): track 0.00 -> 5.83 mm
- net Net-(U2-RT): track 0.00 -> 4.09 mm
- net Net-(U2-SS): track 0.00 -> 3.42 mm
- net Net-(U2-VC): track 0.00 -> 2.56 mm
- net Net-(C3-Pad1): track 0.00 -> 2.56 mm
- net Net-(U2-INTVCC): track 0.00 -> 2.28 mm
- added copper zone on In1.Cu, net GND
- added copper zone on In2.Cu, net GND
Other:
- copper layers 2 -> 4

Commit message: fixed ERC
Parts:
- removed TP7: ~, TestPoint:TestPoint_Pad_1.5x1.5mm
- added C58: .1u, Capacitor_SMD:C_0603_1608Metric, F.Cu at (102.0, 78.0)
- added R39: 620, Resistor_SMD:R_0805_2012Metric, F.Cu at (94.0, 92.5)
- added R40: 620, Resistor_SMD:R_0805_2012Metric, F.Cu at (97.0, 92.5)
- added R41: 620, Resistor_SMD:R_0805_2012Metric, F.Cu at (100.0, 92.5)
- added R42: 620, Resistor_SMD:R_0805_2012Metric, F.Cu at (102.9, 92.5)
- added R43: 620, Resistor_SMD:R_0805_2012Metric, F.Cu at (105.8, 92.5)
- added R44: 620, Resistor_SMD:R_0805_2012Metric, F.Cu at (109.5, 92.7)
- added R45: 620, Resistor_SMD:R_0805_2012Metric, F.Cu at (112.4, 92.7)
- added R46: 620, Resistor_SMD:R_0805_2012Metric, F.Cu at (115.3, 92.7)
- added R47: 620, Resistor_SMD:R_0805_2012Metric, F.Cu at (118.3, 92.7)
- added R48: 620, Resistor_SMD:R_0805_2012Metric, F.Cu at (121.2, 92.7)
- moved C57 57.1 mm to (137.0, 80.0)
- moved C20 51.0 mm to (165.0, 78.7), turned to -90 degrees
- moved CR2 36.5 mm to (152.0, 78.5)
- moved J1 19.9 mm to (95.6, 99.5), turned to 90 degrees
- moved C29 14.5 mm to (132.6, 94.7)
- moved C12 14.2 mm to (142.0, 44.0), turned to -90 degrees
- moved L3 14.0 mm to (139.0, 40.5), turned to 180 degrees
- moved C11 13.5 mm to (136.5, 44.0), turned to 90 degrees
- moved L5 10.9 mm to (140.8, 94.7)
- moved U9 10.9 mm to (143.8, 83.7)
- moved U5 10.9 mm to (133.6, 84.7)
- moved C23 10.9 mm to (151.9, 90.1)
- moved U7 4.61 mm to (102.5, 84.0)
Connections:
- C26 pad 1: Net-(U8-SET) -> Net-(U3-SET)
- C7 pad 1: Net-(U3-SET) -> Net-(U8-SET)
- R15 pad 1: Net-(U8-SET) -> Net-(U3-SET)
- R16 pad 2: Net-(U8-PGFB) -> Net-(U3-PGFB)
- R17 pad 1: Net-(U8-PGFB) -> Net-(U3-PGFB)
- R24 pad 1: Net-(U3-SET) -> Net-(U8-SET)
- R5 pad 2: Net-(U3-PGFB) -> Net-(U8-PGFB)
- R6 pad 1: Net-(U3-PGFB) -> Net-(U8-PGFB)
- R7 pad 1: Net-(U3-SET) -> Net-(U8-SET)
- U3 pad 10: +7V -> +3.3V
- U3 pad 11: +7V -> +3.3V
- U3 pad 12: +7V -> +3.3V
- U7 pad 1: Net-(J1-Pin_1) -> Net-(U7-A1/AH1)
- U7 pad 10: Net-(J1-Pin_10) -> Net-(U7-A8/AH8)
- U7 pad 2: Net-(J1-Pin_2) -> Net-(U7-A2/AH2)
- U7 pad 3: Net-(J1-Pin_3) -> Net-(U7-A3/AH3)
- U7 pad 4: Net-(J1-Pin_4) -> Net-(U7-A4/AH4)
- U7 pad 5: Net-(J1-Pin_5) -> Net-(R43-Pad2)
- U7 pad 6: Net-(J1-Pin_6) -> Net-(R44-Pad2)
- U7 pad 7: Net-(J1-Pin_7) -> Net-(U7-A5/AH5)
- U7 pad 8: Net-(J1-Pin_8) -> Net-(U7-A6/AH6)
- U7 pad 9: Net-(J1-Pin_9) -> Net-(U7-A7/AH7)
- U8 pad 10: +3.3V -> +7V
- U8 pad 11: +3.3V -> +7V
- U8 pad 12: +3.3V -> +7V
Routing:
- net Net-(U7-A8/AH8): track 0.00 -> 18.0 mm
- net /7.526v: track 7.93 -> 24.7 mm, vias 0 -> 3
- net Net-(U7-A7/AH7): track 0.00 -> 16.2 mm
- net /opto4: track 0.00 -> 14.5 mm, vias 0 -> 1
- net /opto7: track 0.00 -> 13.9 mm
- net Net-(U7-A6/AH6): track 0.00 -> 13.8 mm
- net /opto0: track 0.00 -> 13.4 mm
- net /opto3: track 0.00 -> 13.3 mm, vias 0 -> 1
- net /opto6: track 0.00 -> 12.8 mm
- net /opto1: track 0.00 -> 12.6 mm
- net Net-(U7-A5/AH5): track 0.00 -> 11.5 mm
- net /opto5: track 0.00 -> 11.0 mm
- net /opto2: track 0.00 -> 10.8 mm
- net Net-(R44-Pad2): track 0.00 -> 9.43 mm
- net Net-(U7-A1/AH1): track 0.00 -> 7.64 mm
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
Commit message: supplies
Parts:
- added C59: 10u, Capacitor_SMD:C_1206_3216Metric, F.Cu at (145.5, 43.5)
- added C60: 10u, Capacitor_SMD:C_1206_3216Metric, F.Cu at (155.5, 85.5)
- added C61: 10u, Capacitor_SMD:C_1206_3216Metric, F.Cu at (150.5, 66.5)
- moved TP10 175.7 mm to (202.4, 110.0)
- moved TP11 175.7 mm to (202.4, 113.5)
- moved TP12 175.7 mm to (202.4, 117.1)
- moved TP13 175.7 mm to (202.4, 120.7)
- moved TP14 175.7 mm to (202.4, 124.2)
- moved TP29 175.7 mm to (213.1, 102.9)
- moved TP30 175.7 mm to (213.1, 106.5)
- moved TP31 175.7 mm to (213.1, 110.0)
- moved TP32 175.7 mm to (213.1, 113.5)
- moved TP33 175.7 mm to (213.1, 117.1)
- moved TP8 175.7 mm to (202.4, 102.9)
- moved TP9 175.7 mm to (202.4, 106.5)
- moved TP1 175.7 mm to (198.8, 102.9)
- moved TP15 175.7 mm to (205.9, 102.9)
- moved TP16 175.7 mm to (205.9, 106.5)
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Connections:
- C12 pad 1: +5V -> /in7
- C13 pad 1: Net-(U5-EN/UVLO) -> +5V
- C21 pad 1: +5V -> /in3
- C22 pad 1: Net-(U4-SET) -> GND
- C22 pad 2: Net-(C22-Pad2) -> Net-(U4-SET)
- L3 pad 1: +5V -> /in7
- L4 pad 1: +5V -> /in3
- R12 pad 2: Net-(C22-Pad2) -> Net-(U4-SET)
- TP8 pad 1: +5V -> /in3
- U4 pad 1: +5V -> /in3
- U4 pad 13: +5V -> /in3
- U4 pad 2: +5V -> /in3
- U4 pad 3: +5V -> /in3
- U5 pad 1: Net-(U5-EN/UVLO) -> +5V
- U8 pad 1: +5V -> /in7
- U8 pad 2: +5V -> /in7
- U8 pad 3: +5V -> /in7
- U8 pad 4: +5V -> /in7
Routing:
- net +5V: track 61.3 -> 171.3 mm, vias 8 -> 13
- net +3.3VP: track 3.93 -> 112.3 mm, vias 0 -> 2
- net GND: track 34.9 -> 134.2 mm, vias 15 -> 56
- net /-3.76v: track 0.00 -> 41.0 mm, vias 0 -> 4
- net /2.959v: track 0.00 -> 29.3 mm
- net /.3366v: track 0.00 -> 27.3 mm
- net +3.3V: track 0.00 -> 25.2 mm, vias 0 -> 2
- net Net-(U8-PGFB): track 0.00 -> 18.6 mm, vias 0 -> 2
- net +7V: track 0.00 -> 18.0 mm
- net /7.526v: track 24.7 -> 40.5 mm, vias 3 -> 4
- net /in7: track 0.00 -> 14.3 mm
- net Net-(U4-PGFB): track 0.00 -> 12.3 mm, vias 0 -> 2
- net Net-(U5-SW): track 0.00 -> 11.5 mm
- net /in3: track 0.00 -> 10.9 mm
- net Net-(U5-FBX): track 0.00 -> 8.19 mm
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
Commit message: ADC
Parts:
- removed J5, J6, J7, J8, J9: Conn_01x04_Pin, Connector_PinHeader_2.54mm:PinHeader_1x04_P2.54mm_Vertical
- removed TP17, TP18, TP19, TP20, TP30, TP31: ~, TestPoint:TestPoint_Pad_1.5x1.5mm
- added C62: .1u, Capacitor_SMD:C_0603_1608Metric, F.Cu at (169.2, 71.7)
- J2, J3: value Conn_01x04_Pin -> Conn_01x08_Pin; footprint Connector_PinHeader_2.54mm:PinHeader_1x04_P2.54mm_Vertical -> Connector_PinSocket_2.54mm:PinSocket_1x08_P2.54mm_Vertical
- moved TP21 128.7 mm to (110.0, 38.5)
- moved TP28 127.8 mm to (110.0, 44.0)
- moved TP14 116.5 mm to (117.0, 45.0)
- moved TP16 96.8 mm to (136.5, 39.0)
- moved D16 95.1 mm to (193.4, 60.5)
- moved C48 95.0 mm to (182.4, 63.5), turned to 180 degrees
- moved D14 91.3 mm to (199.4, 63.4)
- moved C52 90.6 mm to (182.4, 61.0), turned to 0 degrees
- moved D15 90.1 mm to (193.4, 55.5)
- moved C54 89.0 mm to (187.4, 62.0)
- moved C46 88.7 mm to (182.4, 58.5), turned to 180 degrees
- moved TP32 87.1 mm to (150.0, 53.5)
- moved D2 86.8 mm to (193.4, 65.4)
- moved D13 85.9 mm to (199.4, 58.4)
- moved TP6 85.8 mm to (145.5, 53.5)
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Connections:
- net /.3366v renamed /REFIN1(-)
- net /2.959v renamed /REFIN1(+)
- net Net-(U1A-*CS) renamed /*CS
- net Net-(U1A-DIN) renamed /DIN
- net Net-(U1A-DOUT/*RDY) renamed /DOUT/*RDY
- net Net-(U1A-SCLK) renamed /SCLK
- D1 pad 3: Net-(D1-COM) -> /AIN15
- D10 pad 3: Net-(D10-COM) -> /AIN5
- D11 pad 3: Net-(D11-COM) -> /AIN6
- D12 pad 3: Net-(D12-COM) -> /AIN4
- D13 pad 3: Net-(D13-COM) -> /AIN3
- D14 pad 3: Net-(D14-COM) -> /AIN1
- D15 pad 3: Net-(D15-COM) -> /AIN2
- D16 pad 3: Net-(D16-COM) -> /AIN0
- D2 pad 3: Net-(D2-COM) -> /AIN14
- D3 pad 3: Net-(D3-COM) -> /AIN13
- D4 pad 3: Net-(D4-COM) -> /AIN12
- D5 pad 3: Net-(D5-COM) -> /AIN11
- D6 pad 3: Net-(D6-COM) -> /AIN9
- D7 pad 3: Net-(D7-COM) -> /AIN10
- D8 pad 3: Net-(D8-COM) -> /AIN8
- D9 pad 2: +3.3V -> unconnected-(D9-K-Pad2)
- D9 pad 3: Net-(D9-COM) -> /AIN7
- J2 pad 1: Net-(D2-COM) -> Net-(J2-Pin_1)
- J2 pad 2: Net-(D1-COM) -> Net-(J2-Pin_2)
- J2 pad 3: -3v -> Net-(J2-Pin_3)
- J2 pad 4: +7V -> Net-(J2-Pin_4)
- J3 pad 1: Net-(D4-COM) -> Net-(J3-Pin_1)
- J3 pad 2: Net-(D3-COM) -> Net-(J3-Pin_2)
- J3 pad 3: -3v -> Net-(J3-Pin_3)
- J3 pad 4: +7V -> Net-(J3-Pin_4)
- J4 pad 1: Net-(D7-COM) -> -3v
- J4 pad 2: Net-(D5-COM) -> -3v
- J4 pad 3: -3v -> +7V
- R21 pad 2: Net-(D1-COM) -> Net-(J2-Pin_8)
- R22 pad 2: Net-(D2-COM) -> Net-(J2-Pin_7)
- R25 pad 2: Net-(D3-COM) -> Net-(J2-Pin_6)
- R26 pad 2: Net-(D4-COM) -> Net-(J2-Pin_5)
- R27 pad 2: Net-(D5-COM) -> Net-(J2-Pin_4)
- R28 pad 2: Net-(D7-COM) -> Net-(J2-Pin_3)
- R29 pad 2: Net-(D6-COM) -> Net-(J2-Pin_2)
- R30 pad 2: Net-(D8-COM) -> Net-(J2-Pin_1)
- R31 pad 2: Net-(D9-COM) -> Net-(J3-Pin_4)
- R32 pad 2: Net-(D11-COM) -> Net-(J3-Pin_3)
- R33 pad 2: Net-(D10-COM) -> Net-(J3-Pin_2)
- R34 pad 2: Net-(D12-COM) -> Net-(J3-Pin_1)
- R35 pad 2: Net-(D13-COM) -> Net-(J3-Pin_8)
- R36 pad 2: Net-(D15-COM) -> Net-(J3-Pin_7)
- R37 pad 2: Net-(D14-COM) -> Net-(J3-Pin_6)
- R38 pad 2: Net-(D16-COM) -> Net-(J3-Pin_5)
- U6 pad 14: Net-(U6-GPIO10) -> unconnected-(U6-GPIO10-Pad14)
- U6 pad 15: Net-(U6-GPIO11) -> unconnected-(U6-GPIO11-Pad15)
- U6 pad 16: Net-(U6-GPIO12) -> unconnected-(U6-GPIO12-Pad16)
- U6 pad 17: Net-(U6-GPIO13) -> unconnected-(U6-GPIO13-Pad17)
- U6 pad 19: Net-(U6-GPIO14) -> unconnected-(U6-GPIO14-Pad19)
- U6 pad 20: Net-(U6-GPIO15) -> unconnected-(U6-GPIO15-Pad20)
Routing:
- net +3.3VP: track 112.3 -> 162.9 mm, vias 2 -> 4
- net /DIN: track 0.00 -> 48.0 mm
- net /SCLK: track 0.00 -> 42.5 mm, vias 0 -> 2
- net /*CS: track 0.00 -> 37.8 mm, vias 0 -> 2
- net /DOUT/*RDY: track 0.00 -> 35.7 mm, vias 0 -> 2
- net /AIN1: track 0.00 -> 23.3 mm, vias 0 -> 2
- net /AIN3: track 0.00 -> 20.7 mm, vias 0 -> 2
- net /AIN6: track 0.00 -> 19.8 mm, vias 0 -> 2
- net /REFIN1(+): track 29.3 -> 9.97 mm
- net GND: track 134.2 -> 152.8 mm, vias 56 -> 98
- net /AIN7: track 0.00 -> 18.1 mm, vias 0 -> 2
- net /AIN15: track 0.00 -> 18.1 mm, vias 0 -> 2
- net /AIN2: track 0.00 -> 18.0 mm, vias 0 -> 2
- net /AIN5: track 0.00 -> 16.6 mm, vias 0 -> 2
- net /AIN0: track 0.00 -> 15.6 mm, vias 0 -> 2
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
Commit message: full pcb
Parts:
- added J5: Conn_01x01_Pin, Connector_PinHeader_2.54mm:PinHeader_1x01_P2.54mm_Vertical, F.Cu at (207.0, 88.5)
- J4: value Conn_01x04_Pin -> Conn_01x01_Pin; footprint Connector_PinHeader_2.54mm:PinHeader_1x04_P2.54mm_Vertical -> Connector_PinHeader_2.54mm:PinHeader_1x01_P2.54mm_Vertical
- moved J4 54.4 mm to (207.0, 40.2)
- moved TP29 26.8 mm to (151.0, 74.5)
- moved TP15 21.7 mm to (125.0, 83.0)
- moved TP9 17.9 mm to (156.0, 76.5)
- moved J1 5.28 mm to (95.0, 94.2)
- moved TP22 4.26 mm to (165.8, 66.2)
- moved J3 2.64 mm to (212.8, 45.0)
- moved R40 2.43 mm to (96.3, 90.2)
- moved R41 2.43 mm to (99.3, 90.2)
- moved R42 2.43 mm to (102.2, 90.2)
- moved R39 2.43 mm to (93.4, 90.2)
- moved R43 2.43 mm to (105.2, 90.2)
- moved R44 2.43 mm to (108.8, 90.3)
- moved R45 2.43 mm to (111.8, 90.3)
- moved R48 2.43 mm to (120.6, 90.3)
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Connections:
- D9 pad 2: unconnected-(D9-K-Pad2) -> +3.3V
- J4 pad 1: -3v -> +7V
Routing:
- net +3.3V: track 38.8 -> 180.0 mm, vias 2 -> 19
- net /AIN11: track 4.14 -> 78.5 mm, vias 2 -> 3
- net /AIN9: track 3.79 -> 72.0 mm, vias 2 -> 4
- net /AIN8: track 1.65 -> 67.8 mm, vias 0 -> 4
- net /AIN10: track 2.98 -> 68.3 mm, vias 2 -> 4
- net /AIN13: track 2.65 -> 67.4 mm, vias 2 -> 5
- net /AIN12: track 1.65 -> 62.2 mm, vias 1 -> 3
- net /AIN14: track 3.65 -> 59.6 mm, vias 2 -> 3
- net +7V: track 20.5 -> 74.0 mm
- net /AIN15: track 18.1 -> 63.1 mm, vias 2 -> 3
- net -3v: track 12.6 -> 51.5 mm
- net /AIN0: track 15.6 -> 43.4 mm
- net /AIN4: track 15.5 -> 36.4 mm
- net /AIN2: track 18.0 -> 38.9 mm
- net /AIN6: track 19.8 -> 40.7 mm
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- added copper zone on F.Cu, net GND

Commit message: full pcb1
Parts:
- removed TP1, TP10, TP11, TP12, TP13, TP14, TP15, TP16, TP2, TP21, TP23, TP24, TP28, TP29, TP3, TP32, TP33, TP4, TP5, TP6, TP8, TP9: ~, TestPoint:TestPoint_Pad_1.5x1.5mm
- added -3.8v1: ~, TestPoint:TestPoint_Pad_1.5x1.5mm, F.Cu at (144.0, 97.2)
- added -3v1: ~, TestPoint:TestPoint_Pad_1.5x1.5mm, F.Cu at (183.8, 92.5)
- added .33v1: ~, TestPoint:TestPoint_Pad_1.5x1.5mm, F.Cu at (170.2, 76.5)
- added 2.95v1: ~, TestPoint:TestPoint_Pad_1.5x1.5mm, F.Cu at (171.0, 45.5)
- added 33v1: ~, TestPoint:TestPoint_Pad_1.5x1.5mm, F.Cu at (159.5, 74.2)
- added 5v1: ~, TestPoint:TestPoint_Pad_1.5x1.5mm, F.Cu at (125.2, 85.5)
- added 7.5v1: ~, TestPoint:TestPoint_Pad_1.5x1.5mm, F.Cu at (136.5, 39.0)
- added 7v1: ~, TestPoint:TestPoint_Pad_1.5x1.5mm, F.Cu at (164.8, 36.2)
- added CS1: ~, TestPoint:TestPoint_Pad_1.5x1.5mm, F.Cu at (150.0, 53.2)
- added DIN1: ~, TestPoint:TestPoint_Pad_1.5x1.5mm, F.Cu at (157.0, 61.5)
- added DOUT1: ~, TestPoint:TestPoint_Pad_1.5x1.5mm, F.Cu at (154.0, 53.2)
- added FBX3: ~, TestPoint:TestPoint_Pad_1.5x1.5mm, F.Cu at (132.0, 97.8)
- added FBX7: ~, TestPoint:TestPoint_Pad_1.5x1.5mm, F.Cu at (129.8, 46.8)
- added FEF1: ~, TestPoint:TestPoint_Pad_1.5x1.5mm, F.Cu at (155.5, 49.8)
- added PSW1: ~, TestPoint:TestPoint_Pad_1.5x1.5mm, F.Cu at (164.2, 61.2)
- added SCLK1: ~, TestPoint:TestPoint_Pad_1.5x1.5mm, F.Cu at (152.5, 60.0)
- added SYNC1: ~, TestPoint:TestPoint_Pad_1.5x1.5mm, F.Cu at (156.8, 53.2)
- added gnd1: ~, TestPoint:TestPoint_Pad_1.5x1.5mm, F.Cu at (155.8, 89.2)
- added gnd2: ~, TestPoint:TestPoint_Pad_1.5x1.5mm, F.Cu at (176.0, 44.2)
Routing:
- net GND: track 161.0 -> 144.5 mm, vias 98 -> 335
- net Net-(U1A-*SYNC): track 6.11 -> 14.8 mm
- net Net-(U2-FBX): track 7.68 -> 15.3 mm
- net +3.3V: track 180.0 -> 174.8 mm
- net /in3: track 15.0 -> 11.0 mm
- net Net-(U1A-REFOUT): track 6.65 -> 10.5 mm
- net /REFIN1(+): track 9.97 -> 11.2 mm
- net Net-(U1A-PSW): track 11.7 -> 11.2 mm

Commit message: full pcb1
Parts:
- removed -3v1, .33v1, 2.95v1, 7v1: ~, TestPoint:TestPoint_Pad_1.5x1.5mm
- removed U3, U8: LT3045xMSE, Package_SO:MSOP-12-1EP_3x4mm_P0.65mm_EP1.65x2.85mm
- added R49: 300, Resistor_SMD:R_0805_2012Metric, F.Cu at (156.8, 81.0)
- added R50: 10, Resistor_SMD:R_0805_2012Metric, F.Cu at (166.2, 46.5)
- added TP1: ~, TestPoint:TestPoint_Pad_1.5x1.5mm, F.Cu at (173.2, 46.5)
- added TP2: ~, TestPoint:TestPoint_Pad_1.5x1.5mm, F.Cu at (164.5, 42.0)
- added U10: LT3045xDD, Package_DFN_QFN:DFN-10-1EP_3x3mm_P0.5mm_EP1.65x2.38mm, F.Cu at (153.9, 66.4)
- added U11: LT3045xDD, Package_DFN_QFN:DFN-10-1EP_3x3mm_P0.5mm_EP1.65x2.38mm, F.Cu at (153.8, 43.9)
- C1, C13, C17, C19, C2, C24, C27, C59, C60, C61: footprint Capacitor_SMD:C_1206_3216Metric -> Capacitor_SMD:C_0805_2012Metric
- C15, C30, C5, C55, C8, C9: footprint Capacitor_SMD:C_0603_1608Metric -> Capacitor_SMD:C_0402_1005Metric
- C29: footprint Capacitor_SMD:C_0201_0603Metric -> Capacitor_SMD:C_0402_1005Metric
- C3: footprint Capacitor_SMD:C_0402_1005Metric -> Capacitor_SMD:C_0603_1608Metric
- C56: value 68u -> 47u; footprint tant_68u:TAJB_AVX -> Resistor_SMD:R_1206_3216Metric
- J4, J5: value Conn_01x01_Pin -> Pin
- R17: value 110k -> 100k
- R18: value 2.61k -> 240
- R19: value 4.02k -> 430
- R20: value 3.32k -> 10
- R39, R40, R41, R42, R45, R46, R47, R48: value 620 -> 680
- R43: value 620 -> 10k
- R44: value 620 -> 10
- moved R44 76.3 mm to (169.8, 44.5), turned to 0 degrees
- moved R43 51.0 mm to (152.5, 71.0), turned to 0 degrees
- moved R20 8.00 mm to (159.0, 81.0)
- moved C26 6.17 mm to (158.5, 68.0), turned to 0 degrees
- moved R15 5.13 mm to (158.5, 65.8), turned to 0 degrees
- moved C59 5.06 mm to (150.5, 44.2)
- moved C27 3.34 mm to (158.5, 63.5), turned to 0 degrees
- moved R18 2.71 mm to (169.8, 46.5)
- moved 33v1 2.69 mm to (157.0, 75.2)
- moved R12 2.15 mm to (163.8, 87.2), turned to 90 degrees
- moved C22 2.14 mm to (166.0, 85.2)
- moved R17 1.90 mm to (155.2, 70.2), turned to 90 degrees
- moved R16 1.77 mm to (157.8, 71.2)
- moved R19 1.25 mm to (167.0, 43.8)
- moved DIN1 1.00 mm to (157.0, 60.5)
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Connections:
- R16 pad 2: Net-(U3-PGFB) -> Net-(U10-PGFB)
- R17 pad 1: Net-(U3-PGFB) -> Net-(R17-Pad1)
- R17 pad 2: GND -> Net-(U10-PGFB)
- R18 pad 2: /REFIN1(-) -> Net-(R18-Pad2)
- R19 pad 2: /REFIN1(+) -> Net-(R19-Pad2)
- R20 pad 1: /REFIN1(-) -> Net-(R20-Pad1)
- R43 pad 1: Net-(J1-Pin_5) -> GND
- R43 pad 2: Net-(R43-Pad2) -> Net-(R17-Pad1)
- R44 pad 1: Net-(J1-Pin_6) -> Net-(R19-Pad2)
- R44 pad 2: Net-(R44-Pad2) -> /REFIN1(+)
- U6 pad 23: unconnected-(U6-GND-Pad23) -> GND
- U6 pad 3: unconnected-(U6-GND-Pad3) -> GND
- U6 pad 8: unconnected-(U6-GND-Pad8) -> GND
- U7 pad 5: Net-(R43-Pad2) -> Net-(J1-Pin_5)
- U7 pad 6: Net-(R44-Pad2) -> Net-(J1-Pin_6)
Routing:
- net GND: track 144.5 -> 107.4 mm, vias 335 -> 317
- net +3.3V: track 174.8 -> 189.9 mm, vias 19 -> 21
- net /REFIN1(-): track 41.9 -> 53.4 mm, vias 4 -> 3
- net Net-(J1-Pin_6): track 3.45 -> 12.9 mm
- net Net-(R44-Pad2): track 7.65 -> 0.00 mm
- net Net-(J1-Pin_5): track 3.35 -> 9.96 mm
- net /in3: track 11.0 -> 17.1 mm
- net Net-(U10-PGFB): track 0.00 -> 6.10 mm
- net +5V: track 171.3 -> 176.7 mm
- net Net-(U11-PGFB): track 18.6 -> 13.6 mm
- net Net-(U3-PGFB): track 4.73 -> 0.00 mm
- net Net-(R43-Pad2): track 4.61 -> 0.00 mm
- net /in7: track 14.3 -> 18.5 mm
- net +7V: track 74.0 -> 70.8 mm
- net -3v: track 51.5 -> 54.5 mm
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