File: hw_drawings/straingauge.kicad_pcb (KiCad board)
At the start: 4 copper layers, 167 parts, among them J1 Conn_01x10_Pin, J2 Conn_01x08_Pin, J3 Conn_01x08_Pin, J4 Pin, J5 Pin, U1 AD7124-8BCPZ, U10 LT3045xDD, U11 LT3045xDD, U2 LT8333RDD-PBF, U4 LT3094xDD, U5 LT8333RDD-PBF, U6 Pico, U7 SI8380PM-IU, U9 SIT8008BC-83-33E-2.4576

Commit message: finished project
Parts:
- added D17: BAV99, Package_TO_SOT_SMD:SOT-23, F.Cu at (150.2, 75.6)
- added H1: MountingHole_Pad, MountingHole:MountingHole_3.2mm_M3_Pad, F.Cu at (112.2, 81.2)
- added H2: MountingHole_Pad, MountingHole:MountingHole_3.2mm_M3_Pad, F.Cu at (213.4, 94.6)
- added H3: MountingHole_Pad, MountingHole:MountingHole_3.2mm_M3_Pad, F.Cu at (108.8, 35.4)
- added H4: MountingHole_Pad, MountingHole:MountingHole_3.2mm_M3_Pad, F.Cu at (212.8, 35.4)
- added R51: 680, Resistor_SMD:R_0805_2012Metric, F.Cu at (150.6, 45.8)
- added R52: 16k, Resistor_SMD:R_0805_2012Metric, F.Cu at (158.4, 89.4)
- C23: value tdk-1u -> 1u; footprint tdk_1u:CAP_2012_TDK -> Capacitor_SMD:C_0402_1005Metric
- moved J2 17.7 mm to (212.4, 66.9), turned to 0 degrees
- moved -3.8v1 4.74 mm to (142.5, 92.8)
- moved FBX7 4.01 mm to (125.8, 47.0)
- moved FBX3 3.48 mm to (130.8, 94.5)
- moved C2 3.43 mm to (121.5, 37.2), turned to 90 degrees
- moved C24 3.09 mm to (163.8, 83.5)
- moved C1 2.69 mm to (116.8, 39.0), turned to 90 degrees
- moved C59 2.07 mm to (150.2, 42.2), turned to 90 degrees
- moved R5 2.02 mm to (157.5, 39.7)
- moved R6 2.02 mm to (157.5, 35.7)
- moved C17 1.60 mm to (158.2, 42.5)
- moved R48 1.60 mm to (119.0, 90.3)
- moved C18 1.32 mm to (134.0, 85.5)
- moved C23 1.31 mm to (138.2, 88.2)
- moved C10 1.21 mm to (123.5, 37.8), turned to 90 degrees
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Connections:
- net Net-(J2-Pin_1) renamed /AIN8_C
- net Net-(J2-Pin_2) renamed /AIN9_C
- net Net-(J2-Pin_3) renamed /AIN10_C
- net Net-(J2-Pin_4) renamed /AIN11_C
- net Net-(J2-Pin_5) renamed /AIN12_C
- net Net-(J2-Pin_6) renamed /AIN13_C
- net Net-(J2-Pin_7) renamed /AIN14_C
- net Net-(J2-Pin_8) renamed /AIN15_C
- J3 pad 1: Net-(J3-Pin_1) -> /AIN0_C
- J3 pad 2: Net-(J3-Pin_2) -> /AIN1_C
- J3 pad 3: Net-(J3-Pin_3) -> /AIN2_C
- J3 pad 4: Net-(J3-Pin_4) -> /AIN3_C
- J3 pad 5: Net-(J3-Pin_5) -> /AIN4_C
- J3 pad 6: Net-(J3-Pin_6) -> /AIN5_C
- J3 pad 7: Net-(J3-Pin_7) -> /AIN6_C
- J3 pad 8: Net-(J3-Pin_8) -> /AIN7_C
- R31 pad 2: Net-(J3-Pin_4) -> /AIN7_C
- R32 pad 2: Net-(J3-Pin_3) -> /AIN6_C
- R33 pad 2: Net-(J3-Pin_2) -> /AIN5_C
- R34 pad 2: Net-(J3-Pin_1) -> /AIN4_C
- R35 pad 2: Net-(J3-Pin_8) -> /AIN3_C
- R36 pad 2: Net-(J3-Pin_7) -> /AIN2_C
- R37 pad 2: Net-(J3-Pin_6) -> /AIN1_C
- R38 pad 2: Net-(J3-Pin_5) -> /AIN0_C
- U11 pad 5: GND -> Net-(U11-ILIM)
- U4 pad 6: GND -> Net-(U4-ILIM)
Routing:
- net +7V: track 70.8 -> 101.6 mm, vias 0 -> 4
- net -3v: track 54.5 -> 75.2 mm
- net /AIN6_C: track 0.00 -> 20.2 mm
- net /AIN7_C: track 0.00 -> 19.8 mm
- net /AIN0_C: track 0.00 -> 19.2 mm, vias 0 -> 1
- net /AIN1_C: track 0.00 -> 18.6 mm, vias 0 -> 4
- net /AIN8_C: track 6.88 -> 20.8 mm, vias 0 -> 2
- net /AIN15_C: track 6.72 -> 20.3 mm, vias 1 -> 0
- net /AIN14_C: track 8.02 -> 21.2 mm
- net +5V: track 176.7 -> 165.4 mm, vias 13 -> 11
- net /AIN3_C: track 0.00 -> 10.9 mm, vias 0 -> 2
- net /AIN2_C: track 0.00 -> 9.98 mm, vias 0 -> 1
- net /AIN4_C: track 0.00 -> 9.16 mm, vias 0 -> 1
- net /AIN9_C: track 7.07 -> 15.8 mm, vias 0 -> 1
- net Net-(J3-Pin_2): track 8.73 -> 0.00 mm, vias 1 -> 0
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- added copper zone on B.Cu, net GND
Other:
- board outline added: 130.3 x 73.4 mm
- board text added: "A0"
- board text added: "A1"
- board text added: "A10"
- board text added: "A11"
- board text added: "A12"
- board text added: "A13"
- board text added: "A14"
- board text added: "A15"
- board text added: "A2"
- board text added: "A3"
- board text added: "A4"
- board text added: "A5"
- board text added: "A6"
- board text added: "A7"
- board text added: "A8"
- board text added: "A9"
- board text added: "Universiteit Utrecht Faculteit Sociale wetenschappen Boris Cornelis Bergman Mei 2024"
