File: hw_drawings/straingauge.kicad_pcb (KiCad board)
At the start: 4 copper layers, 130.3 x 73.4 mm, 174 parts, among them J1 Conn_01x10_Pin, J2 Conn_01x08_Pin, J3 Conn_01x08_Pin, J4 Pin, J5 Pin, U1 AD7124-8BCPZ, U10 LT3045xDD, U11 LT3045xDD, U2 LT8333RDD-PBF, U4 LT3094xDD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

Commit message: changed bead
Parts:
- removed L2: 742792040, ul_7429:IND_742792040_WRE
- removed L3, L4: NFZ18SM121SN10D, NFZ18SM121SN10D:IND_NFZ18SM121SN10D_MUR
- added FB1: 500 2A, Inductor_SMD:L_1206_3216Metric, F.Cu at (95.8, 39.0)
- added FB2: 120 1A, Inductor_SMD:L_0603_1608Metric, F.Cu at (137.5, 41.5)
- added FB3: 120 1A, Inductor_SMD:L_0603_1608Metric, F.Cu at (151.9, 85.0)
Routing:
- net +5V: track 165.4 -> 164.5 mm
Other:
- board size 130.3 x 73.4 mm -> 130.3 x 75 mm

Commit message: move l5
Parts:
- FB2, FB3: footprint Inductor_SMD:L_0603_1608Metric -> Inductor_SMD:L_0805_2012Metric
- moved 5v1 15.8 mm to (133.0, 99.3), turned to 90 degrees
- moved C16 14.6 mm to (140.5, 97.8), turned to 0 degrees
- moved L5 14.3 mm to (129.0, 81.3), turned to -90 degrees
- moved R9 12.0 mm to (138.0, 96.8), turned to -90 degrees
- moved FBX3 11.2 mm to (142.0, 93.8), turned to 90 degrees
- moved C57 10.2 mm to (142.5, 91.8), turned to 180 degrees
- moved C15 9.60 mm to (136.0, 95.3), turned to -90 degrees
- moved R10 9.31 mm to (142.5, 89.8), turned to 0 degrees
- moved C13 9.00 mm to (132.5, 93.8), turned to 90 degrees
- moved R11 8.76 mm to (142.0, 86.8), turned to -90 degrees
- moved -3.8v1 8.67 mm to (147.4, 85.6), turned to 90 degrees
- moved C19 7.15 mm to (131.0, 88.8), turned to 90 degrees
- moved CR2 6.36 mm to (136.2, 84.1), turned to 180 degrees
- moved R8 5.45 mm to (139.5, 86.8), turned to 90 degrees
- moved C18 5.16 mm to (133.0, 90.6), turned to 90 degrees
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Routing:
- net /-3.76v: track 54.7 -> 46.5 mm, vias 7 -> 2
- net +5V: track 164.5 -> 171.0 mm
- net +3.3VP: track 164.6 -> 159.2 mm
- net GND: track 113.4 -> 114.0 mm, vias 220 -> 328

Commit message: redesign
Parts:
- removed C14: .1u, Capacitor_SMD:C_0603_1608Metric
- removed C16: 1.5n, Capacitor_SMD:C_0603_1608Metric
- removed C23: 1u, Capacitor_SMD:C_0402_1005Metric
- removed C26: 4.7u, Capacitor_SMD:C_0805_2012Metric
- removed C27: 10u, Capacitor_SMD:C_0805_2012Metric
- removed CR2, CR3: PMEG4020EPK_315, PMEG4020EPK-315:DIODE_DFN1608D-2_NEX
- removed R15: 33k, Resistor_SMD:R_0805_2012Metric
- removed R16: 1M, Resistor_SMD:R_0805_2012Metric
- removed R17: 100k, Resistor_SMD:R_0805_2012Metric
- removed R3: 68k, Resistor_SMD:R_0805_2012Metric
- removed R4, R8: 20k, Resistor_SMD:R_0805_2012Metric
- removed R43: 10k, Resistor_SMD:R_0805_2012Metric
- removed R9: 39k, Resistor_SMD:R_0805_2012Metric
- removed U10: LT3045xDD, Package_DFN_QFN:DFN-10-1EP_3x3mm_P0.5mm_EP1.65x2.38mm
- added D18: 1N5819WS, Diode_SMD:D_SOD-323, F.Cu at (117.8, 41.3)
- added D19: 1N5819WS, Diode_SMD:D_SOD-323, F.Cu at (134.4, 81.5)
- added U3: LT8330ES6, lt8330:TSOT-23_S6_LIT, F.Cu at (135.7, 87.3)
- C3: value 680p -> 1u; footprint Capacitor_SMD:C_0603_1608Metric -> Capacitor_SMD:C_0402_1005Metric
- C4: value .1u -> 1u; footprint Capacitor_SMD:C_0603_1608Metric -> Capacitor_SMD:C_0402_1005Metric
- H1, H2, H3, H4: footprint MountingHole:MountingHole_3.2mm_M3_Pad -> MountingHole:MountingHole_2.2mm_M2
- U2: value LT8333RDD-PBF -> LT8330ES6; footprint LT83333:05-08-1699_ADI -> lt8330:TSOT-23_S6_LIT
- U5: value LT8333RDD-PBF -> AMS1117-3.3; footprint LT83333:05-08-1699_ADI -> Package_TO_SOT_SMD:SOT-223-3_TabPin2
- moved C3 52.6 mm to (164.0, 65.2), turned to 90 degrees
- moved C4 43.4 mm to (135.5, 84.3), turned to 90 degrees
- moved J3 39.2 mm to (212.0, 84.5), turned to 180 degrees
- moved U5 31.7 mm to (158.8, 67.9), turned to 0 degrees
- moved H1 25.5 mm to (94.0, 99.0)
- moved D12 23.6 mm to (195.0, 74.0)
- moved D11 23.5 mm to (195.0, 68.9)
- moved D15 23.5 mm to (195.0, 78.9)
- moved D16 23.5 mm to (195.0, 83.9)
- moved R32 23.5 mm to (205.5, 69.0)
- moved R34 23.5 mm to (205.5, 74.0)
- moved R36 23.5 mm to (205.5, 79.0)
- moved R38 23.5 mm to (205.5, 84.0)
- moved C41 23.3 mm to (186.1, 69.0)
- moved C43 23.3 mm to (186.1, 74.0)
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Connections:
- C15 pad 1: Net-(U5-INTVCC) -> GND
- C15 pad 2: GND -> Net-(U3-INTVCC)
- C3 pad 1: Net-(C3-Pad1) -> +3.3V
- C30 pad 1: +3.3VP -> +3.3V
- C4 pad 1: Net-(U2-SS) -> Net-(U3-SW)
- C4 pad 2: GND -> Net-(D19-A)
- C5 pad 1: Net-(U2-INTVCC) -> GND
- C5 pad 2: GND -> Net-(U2-INTVCC)
- C57 pad 2: Net-(U5-FBX) -> Net-(U3-FBX)
- FBX3 pad 1: Net-(U5-FBX) -> Net-(U3-FBX)
- L1 pad 1: Net-(U2-SW) -> Net-(D18-A)
- L5 pad 3: Net-(U5-SW) -> Net-(U3-SW)
- L5 pad 4: Net-(C23-Pad2) -> Net-(D19-A)
- R10 pad 1: Net-(U5-FBX) -> Net-(U3-FBX)
- R11 pad 2: Net-(U5-FBX) -> Net-(U3-FBX)
- U1 pad 2: +3.3VP -> +3.3V
- U2 pad 1: +5V -> Net-(D18-A)
- U2 pad 2: +5V -> GND
- U2 pad 3: Net-(U2-INTVCC) -> Net-(U2-FBX)
- U2 pad 4: GND -> +5V
- U2 pad 5: Net-(U2-VC) -> Net-(U2-INTVCC)
- U2 pad 6: Net-(U2-FBX) -> +5V
- U5 pad 1: +5V -> GND
- U5 pad 2: +5V -> +3.3V
- U5 pad 3: Net-(U5-INTVCC) -> +5V
Routing:
- net +5V: track 171.0 -> 66.4 mm, vias 11 -> 13
- net GND: track 114.0 -> 31.6 mm, vias 328 -> 235
- net +3.3VP: track 159.2 -> 106.1 mm, vias 4 -> 2
- net /AIN11: track 77.3 -> 29.8 mm, vias 3 -> 0
- net /AIN9: track 72.0 -> 25.7 mm, vias 6 -> 0
- net /AIN8: track 69.3 -> 26.0 mm, vias 4 -> 0
- net /AIN10: track 66.1 -> 26.3 mm, vias 4 -> 0
- net /AIN13: track 65.0 -> 34.4 mm, vias 5 -> 0
- net /-3.76v: track 46.5 -> 18.5 mm, vias 2 -> 8
- net /REFIN1(-): track 51.0 -> 78.9 mm, vias 2 -> 3
- net /AIN12: track 58.9 -> 32.7 mm, vias 4 -> 0
- net /AIN15: track 63.1 -> 37.8 mm, vias 3 -> 0
- net /AIN14: track 59.6 -> 36.3 mm, vias 3 -> 0
- net /7.526v: track 41.6 -> 19.1 mm, vias 2 -> 6
- net /REFIN1(+): track 10.3 -> 29.9 mm, vias 0 -> 2
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- added copper zone on B.Cu, net +5V
- added copper zone on B.Cu, net /-3.76v
- added copper zone on F.Cu, net /-3.76v
- added copper zone on B.Cu, net /7.526v
